File: breakout-board-attiny/breakout-board-attiny.kicad_pcb (KiCad board)
At the start: 2 copper layers, 6 parts, among them J1 Conn_01x07_Male, J2 Conn_01x07_Male, U1 ATtiny424-X

Commit message: Das atTiny breajout board ist fertig!
Laci hat einige Dinge an den breakout boards geändert
Parts:
- J1, J2: footprint Connector_PinHeader_2.54mm:PinHeader_1x07_P2.54mm_Vertical -> Connector_PinSocket_2.54mm:PinSocket_1x07_P2.54mm_Vertical; moved to B.Cu
- moved J1 0.13 mm to (147.0, 112.6), turned to 0 degrees
- moved J2 0.12 mm to (131.5, 112.7), turned to 0 degrees
Other:
- board outline added: 36 x 21.5 mm
- board text added: "GND"
- board text added: "PA1"
- board text added: "PA2"
- board text added: "PA3"
- board text added: "PA4"
- board text added: "PA5"
- board text added: "PA6"
- board text added: "PA7"
- board text added: "PB0/TX/RX"
- board text added: "PB1/XCK"
- board text added: "PB2/TxD"
- board text added: "PB3/RxD"
- board text added: "RESET-UPDI"
- board text added: "VCC"
- board text removed: "PB2/TxD PB3/RxD PA7 PA6 PA5 PA4 5V"
