File: breakout-board-funk/breakout-board-receiver/breakout-board-receiver.kicad_pcb (KiCad board)
At the start: 2 copper layers, 42 x 39.4 mm, 5 parts, among them J1 Conn_01x02_Socket, J3 Conn_01x08_Socket, U1 Si4463_eigen

Commit message: funk breakout board finished and sent out for manufacturing
Routing:
- net GND: track 4.41 -> 72.2 mm
- net /nSEL: track 28.2 -> 63.2 mm
- net /nIRQ: track 27.0 -> 58.3 mm
- net /SDN: track 44.9 -> 61.6 mm
- net /Antenne: track 4.40 -> 2.40 mm
- net +5V: track 26.9 -> 25.9 mm
- net /GPIO0: track 16.6 -> 17.6 mm
- net /GPIO1: track 8.04 -> 8.88 mm
- removed copper zone on F.Cu, net GND
Other:
- board size 42 x 39.4 mm -> 44.2 x 41.2 mm
- board text added: "+5V"
- board text added: "GND"
- board text added: "GPIO0"
- board text added: "GPIO1"
- board text added: "SCLK"
- board text added: "SDI"
- board text added: "SDN"
- board text added: "SDO"
- board text added: "nIRQ"
- board text added: "nSEL"
