File: breakout-board-funk/breakout-board-receiver/breakout-board-receiver.kicad_pcb (KiCad board)
At the start: 2 copper layers, 44.2 x 41.2 mm, 5 parts, among them J1 Conn_01x02_Socket, J3 Conn_01x08_Socket, U1 Si4463_eigen

Commit message: ...
Parts:
- added J2: Conn_01x02_Socket, Connector_JST:JST_EH_B2B-EH-A_1x02_P2.50mm_Vertical, F.Cu at (187.4, 84.0)
- C3, C4, U1: moved to B.Cu
- J1, J3: moved to F.Cu
- moved C4 37.0 mm to (156.0, 85.0)
- moved J1 33.0 mm to (158.0, 95.0), turned to 180 degrees
- moved J3 33.0 mm to (191.0, 112.7), turned to 180 degrees
- moved C3 28.2 mm to (160.4, 85.0)
- moved U1 0.97 mm to (174.9, 97.4)
Connections:
- U1 pad 10: GND -> /gnd
- U1 pad 11: /NC -> /NC_3
- U1 pad 3: /NC -> /NC_1
- U1 pad 4: /NC -> /NC_2
Routing:
- net GND: track 72.2 -> 47.6 mm, vias 1 -> 0
- net /NC: track 19.4 -> 0.00 mm
- net /gnd: track 0.00 -> 2.96 mm
- net /nIRQ: track 58.3 -> 55.9 mm
- net /Antenne: track 2.40 -> 2.85 mm, vias 1 -> 0
- added copper zone on B.Cu, net (none)
Other:
- board size 44.2 x 41.2 mm -> 41.6 x 43.6 mm
- board text added: "LoRasender 4BHEL"

Commit message: ...
Other:
- board size 41.6 x 43.6 mm -> 41.4 x 43.6 mm
- board text added: "LoRamodul 4BHEL"
- board text removed: "LoRasender 4BHEL"
Changed lines of the file:
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@@
       (net 4 "/SCLK") (pinfunction "SCLK") (pintype "input") (thermal_bridge_angle 45))
   )
-  (gr_rect (start 154.8 75.4) (end 196.4 119)
+  (gr_rect (start 152.8 75.2) (end 194.2 118.8)
     (stroke (width 0.1) (type default)) (fill none) (layer "Edge.Cuts"))
-  (gr_text "LoRasender 4BHEL" (at 196.4 77.8) (layer "B.Cu")
+  (gr_text "LoRamodul 4BHEL" (at 193.6 77.8) (layer "B.Cu")
     (effects (font (size 1.5 1.5) (thickness 0.1875)) (justify left bottom mirror))
   )
@@
     (polygon
       (pts
-        (xy 154.8 77.8)
-        (xy 196.4 77.8)
-        (xy 196.4 119)
-        (xy 154.8 119)
+        (xy 152.8 75.2)
+        (xy 194.2 75.2)
+        (xy 194.2 118.8)
+        (xy 152.8 118.8)
       )
     )

Commit message: ...
Other:
- board size 41.4 x 43.6 mm -> 41.4 x 41.1 mm
- board text added: "Bottom"
- board text added: "Funkmodul 4BHEL"
- board text removed: "LoRamodul 4BHEL"
Changed lines of the file:
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@@
     (pad_to_mask_clearance 0)
     (pcbplotparams
-      (layerselection 0x0001000_7fffffff)
+      (layerselection 0x0001000_fffffffe)
       (plot_on_all_layers_selection 0x0000000_00000000)
       (disableapertmacros false)
@@
     (fp_line (start 5 2.2) (end 5 -1.6)
       (stroke (width 0.1) (type solid)) (layer "F.Fab"))
-    (pad "1" thru_hole roundrect (at 0 0 270) (size 1.7 2) (drill 1) (layers "*.Cu" "*.Mask") (roundrect_rratio 0.147059)
+    (pad "1" thru_hole roundrect (at 0 0 270) (size 1.7 2) (drill 1) (layers "*.Cu" "*.Mask") (roundrect_rratio 0.1470588235)
       (net 11 "/Antenne") (pinfunction "Pin_1") (pintype "passive"))
     (pad "2" thru_hole oval (at 2.5 0 270) (size 1.7 2) (drill 1) (layers "*.Cu" "*.Mask")
@@
       (net 4 "/SCLK") (pinfunction "SCLK") (pintype "input") (thermal_bridge_angle 45))
   )
-  (gr_rect (start 152.8 75.2) (end 194.2 118.8)
+  (gr_rect (start 152.8 77.7) (end 194.2 118.8)
     (stroke (width 0.1) (type default)) (fill none) (layer "Edge.Cuts"))
-  (gr_text "LoRamodul 4BHEL" (at 193.6 77.8) (layer "B.Cu")
+  (gr_text "Bottom" (at 161.5 80.5) (layer "B.Cu")
+    (effects (font (size 1.5 1.5) (thickness 0.1875)) (justify left bottom mirror))
+  )
+  (gr_text "Funkmodul 4BHEL" (at 153.5 118.5 270) (layer "B.Cu")
     (effects (font (size 1.5 1.5) (thickness 0.1875)) (justify left bottom mirror))
   )
@@
     (polygon
       (pts
-        (xy 152.8 75.2)
-        (xy 194.2 75.2)
+        (xy 152.8 77.7)
+        (xy 194.2 77.7)
         (xy 194.2 118.8)
         (xy 152.8 118.8)
