File: breakout-board-funk/breakout-board-receiver/breakout-board-receiver.kicad_sch (KiCad schematic)
At the start: 5 parts, among them J1 Conn_01x02_Socket, J3 Conn_01x08_Socket, U1 Si4463_eigen

Commit message: ...
Parts:
- added J2: Conn_01x02_Socket, Connector_JST:JST_EH_B2B-EH-A_1x02_P2.50mm_Vertical, symbol Connector:Conn_01x02_Socket
Connections:
- net Antenne: now also J2.1 (Pin_1)
- net GND: no longer U1.10 (GND)
- removed net NC: U1.11 (NC), U1.3 (NC), U1.4 (NC)
- new net NC_1: U1.3 (NC)
- new net NC_2: U1.4 (NC)
- new net NC_3: U1.11 (NC)
- new net gnd: J2.2 (Pin_2), U1.10 (GND)
Other:
- note added: "Connector for Antenna"
Changed lines of the file:
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@@
   (junction (at 76.2 27.94) (diameter 0) (color 0 0 0 0)
   )
-  (no_connect (at 82.55 33.02))
-  (no_connect (at 110.49 33.02))
-  (no_connect (at 82.55 35.56))
+  (no_connect (at 81.28 33.02))
+  (no_connect (at 111.76 33.02))
+  (no_connect (at 81.28 35.56))
   (polyline (pts (xy 132.08 15.24) (xy 132.08 60.96))
     (stroke (width 0) (type default))
@@
     (stroke (width 0) (type default))
   )
-  (wire (pts (xy 120.65 30.48) (xy 120.65 53.34))
+  (polyline (pts (xy 173.99 44.45) (xy 173.99 55.88))
+    (stroke (width 0) (type default))
+  )
+  (wire (pts (xy 106.68 33.02) (xy 111.76 33.02))
     (stroke (width 0) (type default))
   )
@@
     (stroke (width 0) (type default))
   )
+  (wire (pts (xy 137.16 50.8) (xy 147.32 50.8))
+    (stroke (width 0) (type default))
+  )
+  (wire (pts (xy 147.32 53.34) (xy 137.16 53.34))
+    (stroke (width 0) (type default))
+  )
   (wire (pts (xy 77.47 40.64) (xy 86.36 40.64))
     (stroke (width 0) (type default))
@@
     (stroke (width 0) (type default))
   )
-  (wire (pts (xy 82.55 35.56) (xy 86.36 35.56))
+  (wire (pts (xy 81.28 35.56) (xy 86.36 35.56))
     (stroke (width 0) (type default))
   )
@@
     (stroke (width 0) (type default))
   )
+  (polyline (pts (xy 134.62 44.45) (xy 134.62 55.88))
+    (stroke (width 0) (type default))
+  )
   (wire (pts (xy 76.2 27.94) (xy 86.36 27.94))
     (stroke (width 0) (type default))
@@
     (stroke (width 0) (type default))
   )
+  (polyline (pts (xy 134.62 55.88) (xy 173.99 55.88))
+    (stroke (width 0) (type default))
+  )
   (wire (pts (xy 77.47 38.1) (xy 86.36 38.1))
     (stroke (width 0) (type default))
   )
+  (wire (pts (xy 16.51 72.39) (xy 25.4 72.39))
+    (stroke (width 0) (type default))
+  )
   (wire (pts (xy 66.04 36.83) (xy 66.04 27.94))
     (stroke (width 0) (type default))
@@
     (stroke (width 0) (type default))
   )
-  (polyline (pts (xy 40.64 71.12) (xy 13.97 71.12))
+  (polyline (pts (xy 40.64 74.93) (xy 13.97 74.93))
     (stroke (width 0) (type default))
   )
@@
     (stroke (width 0) (type default))
   )
-  (wire (pts (xy 106.68 33.02) (xy 110.49 33.02))
-    (stroke (width 0) (type default))
-  )
   (wire (pts (xy 54.61 50.8) (xy 66.04 50.8))
     (stroke (width 0) (type default))
@@
     (stroke (width 0) (type default))
   )
+  (polyline (pts (xy 135.89 44.45) (xy 173.99 44.45))
+    (stroke (width 0) (type default))
+  )
   (polyline (pts (xy 50.8 60.96) (xy 50.8 15.24))
     (stroke (width 0) (type default))
@@
     (stroke (width 0) (type default))
   )
+  (polyline (pts (xy 134.62 44.45) (xy 135.89 44.45))
+    (stroke (width 0) (type default))
+  )
   (wire (pts (xy 135.89 21.59) (xy 144.78 21.59))
     (stroke (width 0) (type default))
   )
-  (polyline (pts (xy 40.64 45.72) (xy 40.64 71.12))
+  (polyline (pts (xy 40.64 45.72) (xy 40.64 74.93))
     (stroke (width 0) (type default))
   )
@@
     (stroke (width 0) (type default))
   )
-  (polyline (pts (xy 13.97 71.12) (xy 13.97 45.72))
+  (polyline (pts (xy 13.97 74.93) (xy 13.97 45.72))
+    (stroke (width 0) (type default))
+  )
+  (polyline (pts (xy 134.62 44.45) (xy 135.89 44.45))
     (stroke (width 0) (type default))
   )
@@
     (stroke (width 0) (type default))
   )
-  (wire (pts (xy 82.55 33.02) (xy 86.36 33.02))
+  (wire (pts (xy 81.28 33.02) (xy 86.36 33.02))
     (stroke (width 0) (type default))
   )
@@
     (effects (font (size 1.27 1.27)) (justify left bottom))
   )
+  (text "Connector for Antenna" (at 135.89 46.99 0)
+    (effects (font (size 1.27 1.27)) (justify left bottom))
+  )
   (label "GPIO0" (at 113.03 35.56 0) (fields_autoplaced)
     (effects (font (size 1.27 1.27)) (justify left bottom))
   )
+  (label "gnd" (at 16.51 72.39 0) (fields_autoplaced)
+    (effects (font (size 1.27 1.27)) (justify left bottom))
+  )
+  (label "gnd" (at 137.16 53.34 0) (fields_autoplaced)
+    (effects (font (size 1.27 1.27)) (justify left bottom))
+  )
   (label "nIRQ" (at 135.89 34.29 0) (fields_autoplaced)
     (effects (font (size 1.27 1.27)) (justify left bottom))
@@
     (effects (font (size 1.27 1.27)) (justify left bottom))
   )
-  (label "NC" (at 110.49 33.02 0) (fields_autoplaced)
+  (label "NC_3" (at 111.76 33.02 0) (fields_autoplaced)
     (effects (font (size 1.27 1.27)) (justify left bottom))
   )
@@
     (effects (font (size 1.27 1.27)) (justify left bottom))
   )
-  (label "NC" (at 82.55 35.56 0) (fields_autoplaced)
-    (effects (font (size 1.27 1.27)) (justify left bottom))
-  )
-  (label "NC" (at 82.55 33.02 0) (fields_autoplaced)
+  (label "gnd" (at 120.65 30.48 0) (fields_autoplaced)
+    (effects (font (size 1.27 1.27)) (justify left bottom))
+  )
+  (label "NC_2" (at 81.28 35.56 0) (fields_autoplaced)
+    (effects (font (size 1.27 1.27)) (justify left bottom))
+  )
+  (label "NC_1" (at 81.28 33.02 0) (fields_autoplaced)
     (effects (font (size 1.27 1.27)) (justify left bottom))
   )
   (label "SDO" (at 113.03 40.64 0) (fields_autoplaced)
+    (effects (font (size 1.27 1.27)) (justify left bottom))
+  )
+  (label "Antenne" (at 137.16 50.8 0) (fields_autoplaced)
     (effects (font (size 1.27 1.27)) (justify left bottom))
   )
@@
         (path "/fcf88253-a5aa-45dc-8ee6-d0d909a2a2d5"
           (reference "C3") (unit 1)
+        )
+      )
+    )
+  )
+  (symbol (lib_id "power:PWR_FLAG") (at 25.4 72.39 270) (unit 1)
+    (in_bom yes) (on_board yes) (dnp no) (fields_autoplaced)
+    (property "Reference" "#FLG03" (at 27.305 72.39 0)
+      (effects (font (size 1.27 1.27)) hide)
+    )
+    (property "Value" "PWR_FLAG" (at 29.21 73.025 90)
+      (effects (font (size 1.27 1.27)) (justify left))
+    )
+    (property "Footprint" "" (at 25.4 72.39 0)
+      (effects (font (size 1.27 1.27)) hide)
+    )
+    (property "Datasheet" "~" (at 25.4 72.39 0)
+      (effects (font (size 1.27 1.27)) hide)
+    )
+    (pin "1")
+    (instances
+      (project "breakout-board-receiver"
+        (path "/fcf88253-a5aa-45dc-8ee6-d0d909a2a2d5"
+          (reference "#FLG03") (unit 1)
         )
       )
@@
     )
   )
-  (symbol (lib_id "power:GND") (at 120.65 53.34 0) (unit 1)
-    (in_bom yes) (on_board yes) (dnp no) (fields_autoplaced)
-    (property "Reference" "#PWR010" (at 120.65 59.69 0)
-      (effects (font (size 1.27 1.27)) hide)
-    )
-    (property "Value" "GND" (at 120.65 58.42 0)
+  (symbol (lib_id "RF:Si4460") (at 96.52 40.64 0) (unit 1)
+    (in_bom yes) (on_board yes) (dnp no) (fields_autoplaced)
+    (property "Reference" "U1" (at 96.52 22.86 0)
       (effects (font (size 1.27 1.27)))
     )
-    (property "Footprint" "" (at 120.65 53.34 0)
-      (effects (font (size 1.27 1.27)) hide)
-    )
-    (property "Datasheet" "" (at 120.65 53.34 0)
-      (effects (font (size 1.27 1.27)) hide)
-    )
-    (pin "1")
-    (instances
-      (project "breakout-board-receiver"
-        (path "/fcf88253-a5aa-45dc-8ee6-d0d909a2a2d5"
-          (reference "#PWR010") (unit 1)
-        )
-      )
-    )
-  )
-  (symbol (lib_id "power:+5V") (at 76.2 21.59 0) (unit 1)
-    (in_bom yes) (on_board yes) (dnp no) (fields_autoplaced)
-    (property "Reference" "#PWR08" (at 76.2 25.4 0)
-      (effects (font (size 1.27 1.27)) hide)
-    )
-    (property "Value" "+5V" (at 76.2 17.78 0)
-      (effects (font (size 1.27 1.27)))
-    )
-    (property "Footprint" "" (at 76.2 21.59 0)
-      (effects (font (size 1.27 1.27)) hide)
-    )
-    (property "Datasheet" "" (at 76.2 21.59 0)
-      (effects (font (size 1.27 1.27)) hide)
-    )
-    (pin "1")
-    (instances
-      (project "breakout-board-receiver"
-        (path "/fcf88253-a5aa-45dc-8ee6-d0d909a2a2d5"
-          (reference "#PWR08") (unit 1)
-        )
-      )
-    )
-  )
-  (symbol (lib_name "Si4460_1") (lib_id "RF:Si4460") (at 96.52 40.64 0) (unit 1)
-    (in_bom yes) (on_board yes) (dnp no) (fields_autoplaced)
-    (property "Reference" "U1" (at 97.79 22.86 0)
-      (effects (font (size 1.27 1.27)))
-    )
-    (property "Value" "Si4463_eigen" (at 97.79 25.4 0)
+    (property "Value" "Si4463_eigen" (at 96.52 25.4 0)
       (effects (font (size 1.27 1.27)))
     )
@@
     (pin "16")
     (pin "2")
-    (pin "21")
     (pin "3")
     (pin "4")
-    (pin "5")
     (pin "5")
     (pin "6")
@@
     )
   )
+  (symbol (lib_id "power:+5V") (at 76.2 21.59 0) (unit 1)
+    (in_bom yes) (on_board yes) (dnp no) (fields_autoplaced)
+    (property "Reference" "#PWR08" (at 76.2 25.4 0)
+      (effects (font (size 1.27 1.27)) hide)
+    )
+    (property "Value" "+5V" (at 76.2 17.78 0)
+      (effects (font (size 1.27 1.27)))
+    )
+    (property "Footprint" "" (at 76.2 21.59 0)
+      (effects (font (size 1.27 1.27)) hide)
+    )
+    (property "Datasheet" "" (at 76.2 21.59 0)
+      (effects (font (size 1.27 1.27)) hide)
+    )
+    (pin "1")
+    (instances
+      (project "breakout-board-receiver"
+        (path "/fcf88253-a5aa-45dc-8ee6-d0d909a2a2d5"
+          (reference "#PWR08") (unit 1)
+        )
+      )
+    )
+  )
   (symbol (lib_id "power:GND") (at 17.78 63.5 0) (unit 1)
     (in_bom yes) (on_board yes) (dnp no) (fields_autoplaced)
@@
         )
       )
+    )
+  )
+  (symbol (lib_id "Connector:Conn_01x02_Socket") (at 152.4 50.8 0) (unit 1)
+    (in_bom yes) (on_board yes) (dnp no) (fields_autoplaced)
+    (property "Reference" "J2" (at 153.67 51.435 0)
+      (effects (font (size 1.27 1.27)) (justify left))
+    )
+    (property "Value" "Conn_01x02_Socket" (at 153.67 53.975 0)
+      (effects (font (size 1.27 1.27)) (justify left))
+    )
+    (property "Footprint" "Connector_JST:JST_EH_B2B-EH-A_1x02_P2.50mm_Vertical" (at 152.4 50.8 0)
+      (effects (font (size 1.27 1.27)) hide)
+    )
+    (property "Datasheet" "~" (at 152.4 50.8 0)
+      (effects (font (size 1.27 1.27)) hide)
+    )
+    (pin "1")
+    (pin "2")
+    (instances
+      (project "breakout-board-receiver"
+        (path "/fcf88253-a5aa-45dc-8ee6-d0d909a2a2d5"
+          (reference "J2") (unit 1)
+        )
+      )
