File: breakout-board-display-brain/breakout-board-display-brain/breakout-board-display-brain.kicad_pcb (KiCad board)
At the start: 2 copper layers, 6 parts, among them J1 Conn_01x15_Socket, J2 Conn_01x15_Socket, J3 Conn_01x16_Female, J4 Conn_01x02_Socket, SW1 RotaryEncoder_Switch

Commit message: ...
Parts:
- added J5: Conn_01x11_Socket, Connector_PinSocket_2.54mm:PinSocket_1x11_P2.54mm_Vertical, F.Cu at (138.4, 37.0)
- moved J4 29.5 mm to (132.4, 37.2)
Connections:
- net +5V renamed /5V
Routing:
- net /Pin_2: track 129.3 -> 107.7 mm
- net /Pin_9: track 78.3 -> 60.5 mm
- net /Pin_1: track 115.8 -> 100.2 mm
- net /Pin_3: track 137.0 -> 124.3 mm
- net /Pin_0: track 99.0 -> 90.4 mm
- net /5V: track 103.4 -> 96.0 mm
- net GND: track 90.5 -> 84.6 mm
- net /Pin_7: track 42.0 -> 39.3 mm
- added copper zone on B.Cu, net GND
- removed copper zone on B.Cu, net (none)

Commit message: finsihed breakout-board.display-brain
fertig fürs Fräsen
Parts:
- removed J5: Conn_01x11_Socket, Connector_PinSocket_2.54mm:PinSocket_1x11_P2.54mm_Vertical
- removed RV1: R_Potentiometer, Potentiometer_THT:Potentiometer_ACP_CA9-V10_Vertical
- J1, J2: value Conn_01x15_Socket -> Conn_01x19_Socket; footprint Connector_PinSocket_2.54mm:PinSocket_1x15_P2.54mm_Vertical -> Connector_PinSocket_2.54mm:PinSocket_1x19_P2.54mm_Vertical
- J3: value Conn_01x16_Female -> Conn_01x02_Socket; footprint Connector_PinSocket_2.54mm:PinSocket_1x16_P2.54mm_Vertical -> Connector_PinSocket_2.54mm:PinSocket_1x02_P2.54mm_Vertical
- J4: value Conn_01x02_Socket -> Conn_01x04_Socket; footprint Connector_PinSocket_2.54mm:PinSocket_1x02_P2.54mm_Vertical -> Connector_PinSocket_2.54mm:PinSocket_1x04_P2.54mm_Vertical
- moved J4 74.9 mm to (170.6, 101.6), turned to 0 degrees
- moved J3 61.3 mm to (170.6, 117.3), turned to 180 degrees
- moved SW1 44.0 mm to (163.8, 82.2)
- moved J2 28.5 mm to (154.5, 77.7), turned to 0 degrees
- moved J1 14.6 mm to (129.1, 77.7)
Connections:
- J1 pad 1: GND -> /3V3
- J1 pad 10: GND -> /IO26
- J1 pad 11: /Pin_8 -> /IO27
- J1 pad 12: /Pin_9 -> /IO14
- J1 pad 13: /5V -> /IO12
- J1 pad 14: /5V -> GND
- J1 pad 15: GND -> /IO13
- J1 pad 2: /3.3V -> /EN
- J1 pad 3: /3.3V -> /SENSOR_VP
- J1 pad 4: /RST -> /SENSOR_VN
- J1 pad 5: GND -> /IO34
- J1 pad 6: /Pin_4 -> /IO35
- J1 pad 7: /Pin_5 -> /IO32
- J1 pad 8: /Pin_6 -> /IO33
- J1 pad 9: /Pin_7 -> /IO25
- J2 pad 1: GND -> /CLK
- J2 pad 10: GND -> /IO5_SS
- J2 pad 11: /Pin_3 -> /IO18_SCK
- J2 pad 12: /Pin_2 -> /IO19_MISO
- J2 pad 13: /Pin_1 -> GND
- J2 pad 14: /Pin_0 -> /IO21_SDA
- J2 pad 15: GND -> /RXD0
- J2 pad 2: GND -> /SD0
- J2 pad 3: /Pin_19 -> /SD1
- J2 pad 4: /Pin_18 -> /IO15
- J2 pad 5: GND -> /IO2
- J2 pad 6: /TX -> /IO0
- J2 pad 7: /RX -> /IO4
- J2 pad 8: GND -> /IO16
- J2 pad 9: /Pin_10 -> /IO17
- J3 pad 1: GND -> +5V
- J3 pad 2: /5V -> GND
- J4 pad 1: /5V -> GND
- J4 pad 2: GND -> +5V
- SW1 pad A: /Pin_7 -> /IO2
- SW1 pad B: /Pin_8 -> /IO0
- SW1 pad S1: /Pin_9 -> /IO4
Routing:
- net /Pin_3: track 124.3 -> 0.00 mm
- net /Pin_2: track 107.7 -> 0.00 mm
- net /Pin_1: track 100.2 -> 0.00 mm
- net /5V: track 96.0 -> 0.00 mm
- net /Pin_0: track 90.4 -> 0.00 mm
- net GND: track 84.6 -> 0.00 mm
- net +5V: track 0.00 -> 62.8 mm
- net /Pin_9: track 60.5 -> 0.00 mm
- net /Pin_8: track 41.6 -> 0.00 mm
- net /Pin_7: track 39.3 -> 0.00 mm
- net /V0: track 35.2 -> 0.00 mm
- net /IO4: track 0.00 -> 26.2 mm
- net /Pin_4: track 20.0 -> 0.00 mm
- net /IO22_SCL: track 0.00 -> 19.9 mm
- net /Pin_5: track 19.7 -> 0.00 mm
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Other:
- board outline added: 55 x 51.5 mm
- board text added: "+5V"
- board text added: "GND"
- board text added: "SCL"
- board text added: "SDA"

Commit message: funk breakout board routed
Parts:
- moved J2 45.9 mm to (154.5, 123.6), turned to 180 degrees
- moved SW1 19.3 mm to (149.1, 69.7), turned to 180 degrees
- moved J3 8.68 mm to (162.0, 118.5)
- moved J4 8.68 mm to (162.0, 102.7)
- moved J1 0.31 mm to (129.0, 78.0)
Routing:
- net /IO2: track 11.7 -> 82.3 mm
- net /IO0: track 10.7 -> 73.8 mm
- net /IO4: track 26.2 -> 51.9 mm
- net +5V: track 62.8 -> 39.7 mm
- net /IO21_SDA: track 17.8 -> 36.6 mm
- net /IO22_SCL: track 19.9 -> 31.3 mm
Other:
- board size 55 x 51.5 mm -> 41 x 68.7 mm

Commit message: Revert "Merge branch 'main' of https://github.com/DominikRzecki/mpm-hardware"
This reverts commit b1fb40005cc6000a652d43f250fbd6541baa0df3, reversing
changes made to 77b873b98367f4cea487d2747d29dc0cf0db4d54.
Parts:
- moved J2 45.9 mm to (154.5, 77.7), turned to 0 degrees
- moved SW1 19.3 mm to (163.8, 82.2), turned to 0 degrees
- moved J3 8.68 mm to (170.6, 117.3)
- moved J4 8.68 mm to (170.6, 101.6)
- moved J1 0.31 mm to (129.1, 77.7)
Routing:
- net /IO2: track 82.3 -> 11.7 mm
- net /IO0: track 73.8 -> 10.7 mm
- net /IO4: track 51.9 -> 26.2 mm
- net +5V: track 39.7 -> 62.8 mm
- net /IO21_SDA: track 36.6 -> 17.8 mm
- net /IO22_SCL: track 31.3 -> 19.9 mm
Other:
- board size 41 x 68.7 mm -> 55 x 51.5 mm
