File: breakout-board-display-brain/breakout-board-display-brain/breakout-board-display-brain.kicad_sch (KiCad schematic)
At the start: 7 parts, among them J1 Conn_01x19_Socket, J2 Conn_01x19_Socket, J3 Conn_01x02_Socket, J4 Conn_01x04_Socket, J5 Conn_01x04_Socket, SW1 RotaryEncoder_Switch, U1 ESP32-WROOM-32

Commit message: Updated PCB layout according to new schematic.(ASM1117-> LM317) (Beidl update)
Parts:
- added R1, R2, R3: 10k, symbol Device:R_Small
Connections:
- net +5V: now also R1.1, R2.1, R3.1
- net IO2: now also R1.2, R2.2
- net IO4: now also R3.2
Changed lines of the file:
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@@
   (junction (at 209.55 40.64) (diameter 0) (color 0 0 0 0)
+  )
+  (junction (at 207.01 30.48) (diameter 0) (color 0 0 0 0)
+  )
+  (junction (at 181.61 30.48) (diameter 0) (color 0 0 0 0)
+  )
+  (junction (at 176.53 30.48) (diameter 0) (color 0 0 0 0)
   )
   (no_connect (at 110.49 54.61))
@@
     (stroke (width 0) (type default))
   )
-  (wire (pts (xy 179.07 30.48) (xy 189.23 30.48))
+  (wire (pts (xy 170.18 30.48) (xy 176.53 30.48))
     (stroke (width 0) (type default))
   )
@@
     (stroke (width 0) (type default))
   )
-  (wire (pts (xy 209.55 20.32) (xy 209.55 30.48))
-    (stroke (width 0) (type default))
-  )
   (wire (pts (xy 105.41 64.77) (xy 105.41 80.01))
     (stroke (width 0) (type default))
@@
     (stroke (width 0) (type default))
   )
-  (wire (pts (xy 179.07 26.67) (xy 179.07 30.48))
-    (stroke (width 0) (type default))
-  )
   (polyline (pts (xy 96.52 105.41) (xy 100.33 105.41))
     (stroke (width 0) (type default))
@@
     (stroke (width 0) (type default))
   )
-  (wire (pts (xy 170.18 26.67) (xy 179.07 26.67))
-    (stroke (width 0) (type default))
-  )
   (wire (pts (xy 82.55 82.55) (xy 88.9 82.55))
     (stroke (width 0) (type default))
@@
     (stroke (width 0) (type default))
   )
+  (wire (pts (xy 207.01 30.48) (xy 204.47 30.48))
+    (stroke (width 0) (type default))
+  )
   (polyline (pts (xy 95.25 105.41) (xy 36.83 105.41))
     (stroke (width 0) (type default))
@@
     (stroke (width 0) (type default))
   )
+  (wire (pts (xy 176.53 20.32) (xy 176.53 24.13))
+    (stroke (width 0) (type default))
+  )
   (polyline (pts (xy 13.97 13.97) (xy 13.97 39.37))
     (stroke (width 0) (type default))
@@
     (stroke (width 0) (type default))
   )
+  (wire (pts (xy 176.53 30.48) (xy 181.61 30.48))
+    (stroke (width 0) (type default))
+  )
   (polyline (pts (xy 100.33 81.28) (xy 100.33 86.36))
     (stroke (width 0) (type default))
   )
+  (wire (pts (xy 181.61 20.32) (xy 181.61 21.59))
+    (stroke (width 0) (type default))
+  )
   (wire (pts (xy 209.55 40.64) (xy 209.55 43.18))
     (stroke (width 0) (type default))
@@
     (stroke (width 0) (type default))
   )
+  (wire (pts (xy 176.53 29.21) (xy 176.53 30.48))
+    (stroke (width 0) (type default))
+  )
   (wire (pts (xy 82.55 52.07) (xy 88.9 52.07))
     (stroke (width 0) (type default))
   )
+  (wire (pts (xy 181.61 30.48) (xy 189.23 30.48))
+    (stroke (width 0) (type default))
+  )
   (wire (pts (xy 82.55 46.99) (xy 88.9 46.99))
     (stroke (width 0) (type default))
   )
-  (wire (pts (xy 209.55 30.48) (xy 204.47 30.48))
+  (wire (pts (xy 212.09 30.48) (xy 207.01 30.48))
     (stroke (width 0) (type default))
   )
@@
     (stroke (width 0) (type default))
   )
+  (wire (pts (xy 181.61 26.67) (xy 181.61 30.48))
+    (stroke (width 0) (type default))
+  )
   (wire (pts (xy 223.52 50.8) (xy 234.95 50.8))
     (stroke (width 0) (type default))
@@
     (stroke (width 0) (type default))
   )
+  (wire (pts (xy 207.01 26.67) (xy 207.01 30.48))
+    (stroke (width 0) (type default))
+  )
   (wire (pts (xy 110.49 62.23) (xy 123.19 62.23))
     (stroke (width 0) (type default))
@@
     (stroke (width 0) (type default))
   )
+  (wire (pts (xy 207.01 20.32) (xy 207.01 21.59))
+    (stroke (width 0) (type default))
+  )
   (wire (pts (xy 107.95 77.47) (xy 123.19 77.47))
     (stroke (width 0) (type default))
@@
     (effects (font (size 1.27 1.27)) (justify left bottom))
   )
-  (text "SW" (at 209.55 17.78 0)
+  (text "SW" (at 212.09 27.94 0)
     (effects (font (size 1.27 1.27)) (justify left bottom))
   )
@@
     (effects (font (size 1.27 1.27)) (justify left bottom))
   )
-  (text "DT\n" (at 170.18 24.13 0)
+  (text "DT\n" (at 170.18 27.94 0)
     (effects (font (size 1.27 1.27)) (justify left bottom))
   )
@@
     (effects (font (size 1.27 1.27)) (justify left bottom))
   )
-  (label "IO4" (at 209.55 20.32 0) (fields_autoplaced)
+  (label "IO4" (at 212.09 30.48 0) (fields_autoplaced)
     (effects (font (size 1.27 1.27)) (justify left bottom))
   )
@@
     (effects (font (size 1.27 1.27)) (justify left bottom))
   )
-  (label "IO2" (at 170.18 26.67 0) (fields_autoplaced)
+  (label "IO2" (at 170.18 30.48 0) (fields_autoplaced)
     (effects (font (size 1.27 1.27)) (justify left bottom))
   )
@@
     )
   )
+  (symbol (lib_id "Device:R_Small") (at 176.53 26.67 0) (unit 1)
+    (in_bom yes) (on_board yes) (dnp no) (fields_autoplaced)
+    (property "Reference" "R1" (at 179.07 26.035 0)
+      (effects (font (size 1.27 1.27)) (justify left))
+    )
+    (property "Value" "10k" (at 179.07 28.575 0)
+      (effects (font (size 1.27 1.27)) (justify left))
+    )
+    (property "Footprint" "" (at 176.53 26.67 0)
+      (effects (font (size 1.27 1.27)) hide)
+    )
+    (property "Datasheet" "~" (at 176.53 26.67 0)
+      (effects (font (size 1.27 1.27)) hide)
+    )
+    (pin "1")
+    (pin "2")
+    (instances
+      (project "breakout-board-display-brain"
+        (path "/860671aa-4c8a-4921-a8d3-0a28e74ec70f"
+          (reference "R1") (unit 1)
+        )
+      )
+    )
+  )
   (symbol (lib_name "GND_1") (lib_id "power:GND") (at 220.98 30.48 0) (unit 1)
     (in_bom yes) (on_board yes) (dnp no) (fields_autoplaced)
@@
     )
   )
+  (symbol (lib_id "Device:R_Small") (at 181.61 24.13 0) (unit 1)
+    (in_bom yes) (on_board yes) (dnp no) (fields_autoplaced)
+    (property "Reference" "R2" (at 184.15 23.495 0)
+      (effects (font (size 1.27 1.27)) (justify left))
+    )
+    (property "Value" "10k" (at 184.15 26.035 0)
+      (effects (font (size 1.27 1.27)) (justify left))
+    )
+    (property "Footprint" "" (at 181.61 24.13 0)
+      (effects (font (size 1.27 1.27)) hide)
+    )
+    (property "Datasheet" "~" (at 181.61 24.13 0)
+      (effects (font (size 1.27 1.27)) hide)
+    )
+    (pin "1")
+    (pin "2")
+    (instances
+      (project "breakout-board-display-brain"
+        (path "/860671aa-4c8a-4921-a8d3-0a28e74ec70f"
+          (reference "R2") (unit 1)
+        )
+      )
+    )
+  )
   (symbol (lib_id "power:+5V") (at 16.51 20.32 0) (unit 1)
     (in_bom yes) (on_board yes) (dnp no) (fields_autoplaced)
@@
         (path "/860671aa-4c8a-4921-a8d3-0a28e74ec70f"
           (reference "#PWR01") (unit 1)
+        )
+      )
+    )
+  )
+  (symbol (lib_id "power:+5V") (at 181.61 20.32 0) (unit 1)
+    (in_bom yes) (on_board yes) (dnp no) (fields_autoplaced)
+    (property "Reference" "#PWR014" (at 181.61 24.13 0)
+      (effects (font (size 1.27 1.27)) hide)
+    )
+    (property "Value" "+5V" (at 181.61 16.51 0)
+      (effects (font (size 1.27 1.27)))
+    )
+    (property "Footprint" "" (at 181.61 20.32 0)
+      (effects (font (size 1.27 1.27)) hide)
+    )
+    (property "Datasheet" "" (at 181.61 20.32 0)
+      (effects (font (size 1.27 1.27)) hide)
+    )
+    (pin "1")
+    (instances
+      (project "breakout-board-display-brain"
+        (path "/860671aa-4c8a-4921-a8d3-0a28e74ec70f"
+          (reference "#PWR014") (unit 1)
         )
       )
@@
     )
   )
+  (symbol (lib_id "power:+5V") (at 176.53 20.32 0) (unit 1)
+    (in_bom yes) (on_board yes) (dnp no) (fields_autoplaced)
+    (property "Reference" "#PWR013" (at 176.53 24.13 0)
+      (effects (font (size 1.27 1.27)) hide)
+    )
+    (property "Value" "+5V" (at 176.53 16.51 0)
+      (effects (font (size 1.27 1.27)))
+    )
+    (property "Footprint" "" (at 176.53 20.32 0)
+      (effects (font (size 1.27 1.27)) hide)
+    )
+    (property "Datasheet" "" (at 176.53 20.32 0)
+      (effects (font (size 1.27 1.27)) hide)
+    )
+    (pin "1")
+    (instances
+      (project "breakout-board-display-brain"
+        (path "/860671aa-4c8a-4921-a8d3-0a28e74ec70f"
+          (reference "#PWR013") (unit 1)
+        )
+      )
+    )
+  )
   (symbol (lib_id "power:GND") (at 209.55 43.18 0) (unit 1)
     (in_bom yes) (on_board yes) (dnp no) (fields_autoplaced)
@@
         (path "/860671aa-4c8a-4921-a8d3-0a28e74ec70f"
           (reference "#PWR03") (unit 1)
+        )
+      )
+    )
+  )
+  (symbol (lib_id "power:+5V") (at 207.01 20.32 0) (unit 1)
+    (in_bom yes) (on_board yes) (dnp no) (fields_autoplaced)
+    (property "Reference" "#PWR015" (at 207.01 24.13 0)
+      (effects (font (size 1.27 1.27)) hide)
+    )
+    (property "Value" "+5V" (at 207.01 16.51 0)
+      (effects (font (size 1.27 1.27)))
+    )
+    (property "Footprint" "" (at 207.01 20.32 0)
+      (effects (font (size 1.27 1.27)) hide)
+    )
+    (property "Datasheet" "" (at 207.01 20.32 0)
+      (effects (font (size 1.27 1.27)) hide)
+    )
+    (pin "1")
+    (instances
+      (project "breakout-board-display-brain"
+        (path "/860671aa-4c8a-4921-a8d3-0a28e74ec70f"
+          (reference "#PWR015") (unit 1)
         )
       )
@@
         )
       )
+    )
+  )
+  (symbol (lib_id "Device:R_Small") (at 207.01 24.13 0) (unit 1)
+    (in_bom yes) (on_board yes) (dnp no) (fields_autoplaced)
+    (property "Reference" "R3" (at 209.55 23.495 0)
+      (effects (font (size 1.27 1.27)) (justify left))
+    )
+    (property "Value" "10k" (at 209.55 26.035 0)
+      (effects (font (size 1.27 1.27)) (justify left))
+    )
+    (property "Footprint" "" (at 207.01 24.13 0)
+      (effects (font (size 1.27 1.27)) hide)
+    )
+    (property "Datasheet" "~" (at 207.01 24.13 0)
+      (effects (font (size 1.27 1.27)) hide)
+    )
+    (pin "1")
+    (pin "2")
+    (instances
+      (project "breakout-board-display-brain"
+        (path "/860671aa-4c8a-4921-a8d3-0a28e74ec70f"
+          (reference "R3") (unit 1)
+        )
+      )
