File: breakout-board-power-measurement/breakout-board-power-measurement/breakout-board-power-measurement.kicad_pcb (KiCad board)
At the start: 2 copper layers, 70.6 x 40.2 mm, 83 parts, among them J1 Screw_Terminal_01x04, J2 Conn_01x09, J3 Conn_01x07, J4 Conn_01x02, U1 MCP3911A0-E-SS, U2 Si8641BA-B-IU, U3 LM317_TO-252, Y1 10M

Commit message: Minor fixes.
Parts:
- C1, C2: footprint Capacitor_SMD:C_1206_3216Metric_Pad1.33x1.80mm_HandSolder -> Capacitor_SMD:C_0805_2012Metric_Pad1.18x1.45mm_HandSolder
- moved C1 0.54 mm to (173.2, 149.5)
- moved C2 0.54 mm to (163.9, 149.5)
Routing:
- net GNDD: track 155.4 -> 158.2 mm

Commit message: Fixed SPI
Parts:
- R7: value 10m -> 50m
Connections:
- J2 pad 2: /SDO_ -> /SDI_
- J2 pad 3: /SDI_ -> /SDO_
- R17 pad 1: /SDI -> /SDO
- R17 pad 2: /SDI_ -> /SDO_
- R21 pad 1: /SDO -> /SDI
- R21 pad 2: /SDO_ -> /SDI_
- TP16 pad 1: /SDO_ -> /SDI_
- TP17 pad 1: /SDI_ -> /SDO_
- U1 pad 19: /SDI -> /SDO
- U1 pad 20: /SDO -> /SDI
- U2 pad 12: /~{RESET}_ -> /SDI_
Routing:
- net /SDI_: track 4.45 -> 17.7 mm
- net /~{RESET}_: track 14.3 -> 4.55 mm
- net /SDO_: track 20.6 -> 22.9 mm
- net /SDO: track 6.28 -> 7.10 mm
- net /SDI: track 7.10 -> 6.28 mm
Changed lines of the file:
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@@
       (net 21 "/~{RESET}_") (pinfunction "Pin_1") (pintype "passive"))
     (pad "2" thru_hole oval (at 0 2.54) (size 1.7 1.7) (drill 1) (layers "*.Cu" "*.Mask")
-      (net 22 "/SDO_") (pinfunction "Pin_2") (pintype "passive"))
+      (net 23 "/SDI_") (pinfunction "Pin_2") (pintype "passive"))
     (pad "3" thru_hole oval (at 0 5.08) (size 1.7 1.7) (drill 1) (layers "*.Cu" "*.Mask")
-      (net 23 "/SDI_") (pinfunction "Pin_3") (pintype "passive"))
+      (net 22 "/SDO_") (pinfunction "Pin_3") (pintype "passive"))
     (pad "4" thru_hole oval (at 0 7.62) (size 1.7 1.7) (drill 1) (layers "*.Cu" "*.Mask")
       (net 24 "/SCK_") (pinfunction "Pin_4") (pintype "passive"))
@@
       (stroke (width 0.1) (type solid)) (layer "F.Fab"))
     (pad "1" smd roundrect (at -1 0) (size 1.2 1.4) (layers "F.Cu" "F.Paste" "F.Mask") (roundrect_rratio 0.2083333333)
-      (net 47 "/SDI") (pintype "passive"))
+      (net 46 "/SDO") (pintype "passive"))
     (pad "2" smd roundrect (at 1 0) (size 1.2 1.4) (layers "F.Cu" "F.Paste" "F.Mask") (roundrect_rratio 0.2083333333)
-      (net 23 "/SDI_") (pintype "passive"))
+      (net 22 "/SDO_") (pintype "passive"))
     (model "${KICAD6_3DMODEL_DIR}/Resistor_SMD.3dshapes/R_0805_2012Metric.wrl"
       (offset (xyz 0 0 0))
@@
         (effects (font (size 1 1) (thickness 0.15)))
     )
-    (fp_text value "10m" (at 0 2.62 90) (layer "F.Fab")
+    (fp_text value "50m" (at 0 2.62 90) (layer "F.Fab")
         (effects (font (size 1 1) (thickness 0.15)))
     )
@@
       (stroke (width 0.05) (type solid)) (fill none) (layer "F.CrtYd"))
     (pad "1" thru_hole circle (at 0 0) (size 1.5 1.5) (drill 0.8) (layers "*.Cu" "*.Mask")
-      (net 22 "/SDO_") (pinfunction "1") (pintype "passive"))
+      (net 23 "/SDI_") (pinfunction "1") (pintype "passive"))
   )
   (footprint "Resistor_SMD:R_1206_3216Metric_Pad1.30x1.75mm_HandSolder" (layer "F.Cu")
@@
       (stroke (width 0.05) (type solid)) (fill none) (layer "F.CrtYd"))
     (pad "1" thru_hole circle (at 0 0) (size 1.5 1.5) (drill 0.8) (layers "*.Cu" "*.Mask")
-      (net 23 "/SDI_") (pinfunction "1") (pintype "passive"))
+      (net 22 "/SDO_") (pinfunction "1") (pintype "passive"))
   )
   (footprint "Via:Via_THTPad_D1.5mm_Drill0.8mm" (layer "F.Cu")
@@
       (stroke (width 0.1) (type solid)) (layer "F.Fab"))
     (pad "1" smd roundrect (at -1 0) (size 1.2 1.4) (layers "F.Cu" "F.Paste" "F.Mask") (roundrect_rratio 0.2083333333)
-      (net 46 "/SDO") (pintype "passive"))
+      (net 47 "/SDI") (pintype "passive"))
     (pad "2" smd roundrect (at 1 0) (size 1.2 1.4) (layers "F.Cu" "F.Paste" "F.Mask") (roundrect_rratio 0.2083333333)
-      (net 22 "/SDO_") (pintype "passive"))
+      (net 23 "/SDI_") (pintype "passive"))
     (model "${KICAD6_3DMODEL_DIR}/Resistor_SMD.3dshapes/R_0805_2012Metric.wrl"
       (offset (xyz 0 0 0))
@@
       (net 44 "/SCK") (pinfunction "SCK") (pintype "input"))
     (pad "19" smd rect (at 3.6322 -2.274999) (size 1.651 0.4318) (layers "F.Cu" "F.Paste" "F.Mask")
-      (net 47 "/SDI") (pinfunction "SDO") (pintype "input"))
+      (net 46 "/SDO") (pinfunction "SDO") (pintype "input"))
     (pad "20" smd rect (at 3.6322 -2.924998) (size 1.651 0.4318) (layers "F.Cu" "F.Paste" "F.Mask")
-      (net 46 "/SDO") (pinfunction "SDI") (pintype "input"))
+      (net 47 "/SDI") (pinfunction "SDI") (pintype "input"))
   )
   (footprint "Via:Via_THTPad_D1.5mm_Drill0.8mm" (layer "F.Cu")
@@
       (net 22 "/SDO_") (pinfunction "B4") (pintype "input"))
     (pad "12" smd roundrect (at 2.475 -0.635 270) (size 1.95 0.6) (layers "B.Cu" "B.Paste" "B.Mask") (roundrect_rratio 0.25)
-      (net 21 "/~{RESET}_") (pinfunction "B3") (pintype "output"))
+      (net 23 "/SDI_") (pinfunction "B3") (pintype "output"))
     (pad "13" smd roundrect (at 2.475 0.635 270) (size 1.95 0.6) (layers "B.Cu" "B.Paste" "B.Mask") (roundrect_rratio 0.25)
       (net 24 "/SCK_") (pinfunction "B2") (pintype "output"))
@@
   (segment (start 183.1594 131.3942) (end 183.1848 131.3688) (width 0.4) (layer "F.Cu") (net 21))
   (segment (start 181.416108 131.3942) (end 183.1594 131.3942) (width 0.4) (layer "F.Cu") (net 21))
-  (segment (start 183.1848 131.3688) (end 182.4228 131.3688) (width 0.4) (layer "B.Cu") (net 21))
   (segment (start 183.1848 131.3688) (end 183.7182 131.3688) (width 0.4) (layer "B.Cu") (net 21))
-  (segment (start 182.4228 131.3688) (end 179.324 128.27) (width 0.4) (layer "B.Cu") (net 21))
-  (segment (start 179.324 128.27) (end 179.324 123.633) (width 0.4) (layer "B.Cu") (net 21))
   (segment (start 184.404 130.683) (end 185.674 130.683) (width 0.4) (layer "B.Cu") (net 21))
   (segment (start 183.7182 131.3688) (end 184.404 130.683) (width 0.4) (layer "B.Cu") (net 21))
-  (segment (start 181.452046 133.939154) (end 183.113554 133.939154) (width 0.4) (layer "F.Cu") (net 22))
-  (segment (start 185.674 133.223) (end 186.9694 133.223) (width 0.4) (layer "B.Cu") (net 22))
-  (segment (start 187.1472 129.286) (end 186.8424 128.9812) (width 0.4) (layer "B.Cu") (net 22))
-  (segment (start 182.626 128.9812) (end 180.594 126.9492) (width 0.4) (layer "B.Cu") (net 22))
-  (segment (start 186.9694 133.223) (end 187.1472 133.0452) (width 0.4) (layer "B.Cu") (net 22))
-  (segment (start 183.1848 133.9342) (end 183.7182 133.9342) (width 0.4) (layer "B.Cu") (net 22))
-  (segment (start 187.1472 133.0452) (end 187.1472 129.286) (width 0.4) (layer "B.Cu") (net 22))
-  (segment (start 184.4294 133.223) (end 185.674 133.223) (width 0.4) (layer "B.Cu") (net 22))
-  (segment (start 186.8424 128.9812) (end 182.626 128.9812) (width 0.4) (layer "B.Cu") (net 22))
-  (segment (start 180.594 126.9492) (end 180.594 123.633) (width 0.4) (layer "B.Cu") (net 22))
-  (segment (start 183.7182 133.9342) (end 184.4294 133.223) (width 0.4) (layer "B.Cu") (net 22))
-  (segment (start 181.477446 136.504554) (end 183.129046 136.504554) (width 0.4) (layer "F.Cu") (net 23))
-  (segment (start 184.4802 135.763) (end 185.674 135.763) (width 0.4) (layer "B.Cu") (net 23))
-  (segment (start 183.1848 136.4996) (end 183.7436 136.4996) (width 0.4) (layer "B.Cu") (net 23))
-  (segment (start 183.7436 136.4996) (end 184.4802 135.763) (width 0.4) (layer "B.Cu") (net 23))
+  (segment (start 181.477446 136.504554) (end 183.129046 136.504554) (width 0.4) (layer "F.Cu") (net 22))
+  (segment (start 187.1472 129.286) (end 187.1472 135.2528) (width 0.4) (layer "B.Cu") (net 22))
+  (segment (start 187.1472 135.2528) (end 186.637 135.763) (width 0.4) (layer "B.Cu") (net 22))
+  (segment (start 184.4802 135.763) (end 185.674 135.763) (width 0.4) (layer "B.Cu") (net 22))
+  (segment (start 180.594 126.9492) (end 182.626 128.9812) (width 0.4) (layer "B.Cu") (net 22))
+  (segment (start 183.1848 136.4996) (end 183.7436 136.4996) (width 0.4) (layer "B.Cu") (net 22))
+  (segment (start 186.637 135.763) (end 185.674 135.763) (width 0.4) (layer "B.Cu") (net 22))
+  (segment (start 182.626 128.9812) (end 186.8424 128.9812) (width 0.4) (layer "B.Cu") (net 22))
+  (segment (start 183.7436 136.4996) (end 184.4802 135.763) (width 0.4) (layer "B.Cu") (net 22))
+  (segment (start 180.594 123.633) (end 180.594 126.9492) (width 0.4) (layer "B.Cu") (net 22))
+  (segment (start 186.8424 128.9812) (end 187.1472 129.286) (width 0.4) (layer "B.Cu") (net 22))
+  (segment (start 181.452046 133.939154) (end 183.113554 133.939154) (width 0.4) (layer "F.Cu") (net 23))
+  (segment (start 183.1848 133.9342) (end 183.7158 133.9342) (width 0.4) (layer "B.Cu") (net 23))
+  (segment (start 179.324 123.633) (end 179.324 132.424) (width 0.4) (layer "B.Cu") (net 23))
+  (segment (start 180.8458 133.9342) (end 183.1848 133.9342) (width 0.4) (layer "B.Cu") (net 23))
+  (segment (start 184.427 133.223) (end 185.674 133.223) (width 0.4) (layer "B.Cu") (net 23))
+  (segment (start 180.84 133.94) (end 180.8458 133.9342) (width 0.4) (layer "B.Cu") (net 23))
+  (segment (start 183.7158 133.9342) (end 184.427 133.223) (width 0.4) (layer "B.Cu") (net 23))
+  (segment (start 179.324 132.424) (end 180.84 133.94) (width 0.4) (layer "B.Cu") (net 23))
   (segment (start 181.477446 139.044554) (end 183.129046 139.044554) (width 0.4) (layer "F.Cu") (net 24))
   (segment (start 183.7436 139.0396) (end 184.4802 138.303) (width 0.4) (layer "B.Cu") (net 24))
@@
   (segment (start 176.687354 144.124554) (end 178.377446 144.124554) (width 0.4) (layer "F.Cu") (net 45))
   (segment (start 172.212 137.500002) (end 173.872802 137.500002) (width 0.4) (layer "F.Cu") (net 45))
-  (segment (start 178.352046 133.939154) (end 174.782354 133.939154) (width 0.4) (layer "F.Cu") (net 46))
-  (segment (start 174.782354 133.939154) (end 174.443202 133.600002) (width 0.4) (layer "F.Cu") (net 46))
-  (segment (start 172.212 133.600002) (end 174.443202 133.600002) (width 0.4) (layer "F.Cu") (net 46))
-  (segment (start 172.212 134.250001) (end 174.244673 134.250001) (width 0.4) (layer "F.Cu") (net 47))
-  (segment (start 176.499226 136.504554) (end 178.377446 136.504554) (width 0.4) (layer "F.Cu") (net 47))
-  (segment (start 174.244673 134.250001) (end 176.499226 136.504554) (width 0.4) (layer "F.Cu") (net 47))
+  (segment (start 172.212 134.250001) (end 174.244673 134.250001) (width 0.4) (layer "F.Cu") (net 46))
+  (segment (start 176.499226 136.504554) (end 178.377446 136.504554) (width 0.4) (layer "F.Cu") (net 46))
+  (segment (start 174.244673 134.250001) (end 176.499226 136.504554) (width 0.4) (layer "F.Cu") (net 46))
+  (segment (start 178.352046 133.939154) (end 174.782354 133.939154) (width 0.4) (layer "F.Cu") (net 47))
+  (segment (start 174.782354 133.939154) (end 174.443202 133.600002) (width 0.4) (layer "F.Cu") (net 47))
+  (segment (start 172.212 133.600002) (end 174.443202 133.600002) (width 0.4) (layer "F.Cu") (net 47))
   (segment (start 176.738154 141.584554) (end 178.377446 141.584554) (width 0.4) (layer "F.Cu") (net 48))
   (segment (start 176.184 141.0304) (end 176.738154 141.584554) (width 0.4) (layer "F.Cu") (net 48))
