File: funk-final/funk-transmitter-final/funk-transmitter-final.kicad_sch (KiCad schematic)
At the start: 7 parts, among them J1 Conn_01x02_Socket, J3 Conn_01x02_Socket, J4 Conn_01x05_Socket, J5 Conn_01x03_Socket, U1 Si4463_eigen

Commit message: display and funk changed
Parts:
- J5: footprint Connector_PinSocket_2.54mm:PinSocket_1x03_P2.54mm_Vertical -> Connector_PinHeader_2.54mm:PinHeader_1x03_P2.54mm_Vertical
Changed lines of the file:
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@@
       (effects (font (size 1.27 1.27)) (justify left))
     )
-    (property "Footprint" "Connector_PinSocket_2.54mm:PinSocket_1x03_P2.54mm_Vertical" (at 153.67 57.15 0)
+    (property "Footprint" "Connector_PinHeader_2.54mm:PinHeader_1x03_P2.54mm_Vertical" (at 153.67 57.15 0)
       (effects (font (size 1.27 1.27)) hide)
     )
