File: display-brain-final/display-brain-final/display-brain-final.kicad_pcb (KiCad board)
At the start: 2 copper layers, 104.2 x 68 mm, 25 parts, among them J1 Conn_01x02_Socket, J2 Conn_01x05_Socket, J3 Conn_01x19_Socket, J4 Conn_01x19_Socket, J5 Conn_01x04_Socket, J6 Conn_01x05_Socket, J7 Conn_01x02_Socket, J8 Conn_01x03_Socket, P1 USB_C_Plug_USB2.0, U3 LM317_TO-252

Commit message: platinen angepasst
Routing:
- added copper zone on In1.Cu, net GND
- added copper zone on In2.Cu, net GND
Other:
- copper layers 2 -> 4
- board text added: "GPIO0"
- board text added: "GPIO1"
- board text added: "SDN"
- board text added: "nIRQ"
- board text added: "nSEL"
- board text removed: "IO0"
- board text removed: "IO2"
Changed lines of the file:
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@@
   (layers
     (0 "F.Cu" signal)
+    (1 "In1.Cu" signal)
+    (2 "In2.Cu" signal)
     (31 "B.Cu" signal)
     (32 "B.Adhes" user "B.Adhesive")
@@
       (layer "F.Mask" (type "Top Solder Mask") (thickness 0.01))
       (layer "F.Cu" (type "copper") (thickness 0.035))
-      (layer "dielectric 1" (type "core") (thickness 1.51) (material "FR4") (epsilon_r 4.5) (loss_tangent 0.02))
+      (layer "dielectric 1" (type "prepreg") (thickness 0.1) (material "FR4") (epsilon_r 4.5) (loss_tangent 0.02))
+      (layer "In1.Cu" (type "copper") (thickness 0.035))
+      (layer "dielectric 2" (type "core") (thickness 1.24) (material "FR4") (epsilon_r 4.5) (loss_tangent 0.02))
+      (layer "In2.Cu" (type "copper") (thickness 0.035))
+      (layer "dielectric 3" (type "prepreg") (thickness 0.1) (material "FR4") (epsilon_r 4.5) (loss_tangent 0.02))
       (layer "B.Cu" (type "copper") (thickness 0.035))
       (layer "B.Mask" (type "Bottom Solder Mask") (thickness 0.01))
@@
     (effects (font (size 1 1) (thickness 0.15)) (justify left bottom))
   )
+  (gr_text "nIRQ" (at 223.7 79.8) (layer "F.SilkS")
+    (effects (font (size 1 1) (thickness 0.15)) (justify left bottom))
+  )
   (gr_text "program" (at 165.2 64.6 90) (layer "F.SilkS")
     (effects (font (size 1 1) (thickness 0.15)) (justify left bottom))
@@
     (effects (font (size 1 1) (thickness 0.15)) (justify left bottom))
   )
+  (gr_text "GPIO1" (at 223.8 74.8) (layer "F.SilkS")
+    (effects (font (size 1 1) (thickness 0.15)) (justify left bottom))
+  )
   (gr_text "RXD" (at 170.3 63.6) (layer "F.SilkS")
     (effects (font (size 1 1) (thickness 0.15)) (justify left bottom))
   )
+  (gr_text "GPIO0" (at 223.7 77.3) (layer "F.SilkS")
+    (effects (font (size 1 1) (thickness 0.15)) (justify left bottom))
+  )
   (gr_text "5V" (at 170.2 88.4) (layer "F.SilkS")
     (effects (font (size 1 1) (thickness 0.15)) (justify left bottom))
@@
     (effects (font (size 1 1) (thickness 0.15)) (justify left bottom))
   )
-  (gr_text "IO0" (at 223.8 94.1) (layer "F.SilkS")
-    (effects (font (size 1 1) (thickness 0.15)) (justify left bottom))
-  )
-  (gr_text "IO2" (at 223.8 83.8) (layer "F.SilkS")
+  (gr_text "SDN" (at 223.8 94.1) (layer "F.SilkS")
+    (effects (font (size 1 1) (thickness 0.15)) (justify left bottom))
+  )
+  (gr_text "nSEL" (at 223.8 83.8) (layer "F.SilkS")
     (effects (font (size 1 1) (thickness 0.15)) (justify left bottom))
   )
@@
   (segment (start 166.17 87.13) (end 168.1 85.2) (width 0.4) (layer "B.Cu") (net 6))
   (segment (start 135.5 77.6) (end 145.03 87.13) (width 0.4) (layer "B.Cu") (net 6))
-  (segment (start 146.12 82.17) (end 146.12 77.05) (width 0.4) (layer "F.Cu") (net 8))
-  (segment (start 146.12 77.05) (end 146.11 77.04) (width 0.4) (layer "F.Cu") (net 8))
   (segment (start 150.615 80.495) (end 147.645 80.495) (width 0.4) (layer "F.Cu") (net 8))
   (segment (start 144.585 87.74) (end 144.585 83.855) (width 0.5) (layer "F.Cu") (net 8))
@@
   (segment (start 151.29 79.82) (end 150.615 80.495) (width 0.4) (layer "F.Cu") (net 8))
   (segment (start 151.29 78.51) (end 151.29 79.82) (width 0.4) (layer "F.Cu") (net 8))
+  (segment (start 146.475 76.288508) (end 146.475 79.325) (width 0.4) (layer "F.Cu") (net 8))
+  (segment (start 146.475 79.325) (end 147.645 80.495) (width 0.4) (layer "F.Cu") (net 8))
   (segment (start 147.675 83.875) (end 147.645 83.845) (width 0.5) (layer "F.Cu") (net 8))
   (segment (start 144.585 83.855) (end 144.595 83.845) (width 0.5) (layer "F.Cu") (net 8))
   (segment (start 147.675 87.7825) (end 147.675 83.875) (width 0.5) (layer "F.Cu") (net 8))
-  (via (at 146.11 77.04) (size 1.2) (drill 0.8) (layers "F.Cu" "B.Cu") (net 8))
-  (segment (start 142.1 77.04) (end 146.11 77.04) (width 0.5) (layer "B.Cu") (net 8))
+  (via (at 146.475 76.288508) (size 1.2) (drill 0.8) (layers "F.Cu" "B.Cu") (net 8))
+  (segment (start 142.1 77.04) (end 145.723508 77.04) (width 0.5) (layer "B.Cu") (net 8))
   (segment (start 139.68 67.06) (end 139.68 74.62) (width 0.5) (layer "B.Cu") (net 8))
+  (segment (start 145.723508 77.04) (end 146.475 76.288508) (width 0.5) (layer "B.Cu") (net 8))
   (segment (start 133.1 60.48) (end 139.68 67.06) (width 0.5) (layer "B.Cu") (net 8))
   (segment (start 139.68 74.62) (end 142.1 77.04) (width 0.5) (layer "B.Cu") (net 8))
@@
       )
     )
+  )
+  (zone (net 3) (net_name "GND") (layers "In1.Cu" "In2.Cu") (hatch edge 0.5)
+    (priority 2)
+    (connect_pads (clearance 0.5))
+    (min_thickness 0.25) (filled_areas_thickness no)
+    (fill yes (thermal_gap 0.5) (thermal_bridge_width 0.5))
+    (polygon
+      (pts
+        (xy 126.1 48.7)
+        (xy 126.1 116.7)
+        (xy 230.3 116.7)
+        (xy 230.3 48.7)
+      )
+    )
