File: power-measurement-final/power-measurement-final/power-measurement-final.kicad_sch (KiCad schematic)
At the start: 88 parts, among them J1 Screw_Terminal_01x04, J2 Conn_01x09, J3 Conn_01x07, J4 Conn_01x02, J5 Conn_01x07_Socket, J6 Conn_01x07_Socket, J7 Conn_01x05_Socket, J8 Conn_01x03_Socket, J9 Conn_01x02_Socket, U1 MCP3911A0-E-SS, U2 Si8641BA-B-IU, U3 LM317_TO-252, Y1 10M

Commit message: power measurement final platine started
Parts:
- removed JP1: Jumper_3_Open, Connector_PinHeader_2.54mm:PinHeader_1x03_P2.54mm_Vertical, symbol Jumper:Jumper_3_Open
- removed TP1, TP10, TP11, TP12, TP13, TP14, TP15, TP16, TP17, TP18, TP19, TP2, TP20, TP21, TP22, TP3, TP4, TP5, TP6, TP7, TP8, TP9: TestPoint, Via:Via_THTPad_D1.5mm_Drill0.8mm, symbol Connector:TestPoint
- removed TP23, TP24: TestPoint, Screwhole:Screwhole_THTPad_D3.0mm_Drill2.0mm, symbol Connector:TestPoint
- J5, J6: footprint (none) -> Connector_PinSocket_2.54mm:PinSocket_1x07_P2.54mm_Vertical
- J7: footprint (none) -> Connector_PinSocket_2.54mm:PinSocket_1x05_P2.54mm_Vertical
- J8: footprint (none) -> Connector_PinSocket_2.54mm:PinSocket_1x03_P2.54mm_Vertical
- J9: footprint (none) -> Connector_PinSocket_2.54mm:PinSocket_1x02_P2.54mm_Vertical
Connections:
- net +3.3V: now also J5.1 (Pin_1)
- net GNDD: now also J6.7 (Pin_7)
- net OSC1: now also U1.15 (OSC1/CLKI)
- net SDI: now also J7.3 (Pin_3)
- net SDO: now also J7.2 (Pin_2)
- net SDA/XCK/PB1: now reaches J6.1 (Pin_1)
- net SCL/XDIR/PB0: now reaches J6.2 (Pin_2)
- net RESET-UDPI: now reaches J6.3 (Pin_3)
- net TXD/PA1: now reaches J6.4 (Pin_4)
- net RXD/PA2: now reaches J6.5 (Pin_5)
- net XCK/PA3: now reaches J6.6 (Pin_6)
- net nIRQ: now reaches J8.1 (Pin_1)
- net GPIO0: now reaches J8.2 (Pin_2)
- net GPIO1: now reaches J8.3 (Pin_3)
- net nSEL: now reaches J7.1 (Pin_1)
- net SCLK: now reaches J7.4 (Pin_4)
- net SDN: now reaches J7.5 (Pin_5)
- net Antenne: now reaches J9.1 (Pin_1)
- net XDIR/PA4: now reaches J5.2 (Pin_2)
- net PA5: now reaches J5.3 (Pin_3)
- net PA6: now reaches J5.4 (Pin_4)
- net PA7: now reaches J5.5 (Pin_5)
- net RxD/PB3: now reaches J5.6 (Pin_6)
- net TxD/PB2: now reaches J5.7 (Pin_7)
- no-connect marks 4 -> 3
Other:
- moved on the sheet: C1, C10, C11, C12, C13, C14, C15, C16, C2, C3, C4, C5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

Commit message: power measuremnt final weitergemacht
Parts:
- added D3: LED, Diode_SMD:D_1206_3216Metric_Pad1.42x1.75mm_HandSolder, symbol Device:LED
- added J10: Conn_01x03_Socket, Connector_PinSocket_2.54mm:PinSocket_1x03_P2.54mm_Vertical, symbol Connector:Conn_01x03_Socket
- added R26: 330, Resistor_SMD:R_1206_3216Metric_Pad1.30x1.75mm_HandSolder, symbol Device:R
- added TP1, TP2, TP3, TP4: TestPoint, TestPoint:TestPoint_Plated_Hole_D3.0mm, symbol Connector:TestPoint
Connections:
- net SDO is gone; now on net RXD/PA2: J7.2 (Pin_2), R17.1, U1.19 (SDO)
- net TXD/PA1 is gone; now on net SDI: J6.4 (Pin_4)
- net XCK/PA3 is gone; now on net SCLK: J6.6 (Pin_6)
- net nSEL is gone; now on net PA6: J7.1 (Pin_1)
- net GNDD: now also J9.2 (Pin_2), D3.1 (K)
- net PA5: now also R26.1
- net RESET-UDPI: now also J10.1 (Pin_1)
- net RxD/PB3: now also J10.2 (Pin_2)
- net TxD/PB2: now also J10.3 (Pin_3)
- net Antenne renamed +5V
- new net: D3.2 (A), R26.2
- no-connect marks 3 -> 6
Other:
- note added: "ATtiny programming pins"
- note added: "Schraubbefestigungen"
- note added: "Status LED"
- moved on the sheet: C3, C4, C5, C6, J7, J8, J9, L2, L3, R10, R11, R12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

Commit message: finales power measurement modul weitergemacht
Parts:
- removed J2: Conn_01x09, Connector_PinHeader_2.54mm:PinHeader_1x09_P2.54mm_Vertical, symbol Connector_Generic:Conn_01x09
- removed J3: Conn_01x07, Connector_PinHeader_2.54mm:PinHeader_1x07_P2.54mm_Vertical, symbol Connector_Generic:Conn_01x07
- removed J4: Conn_01x02, Connector_PinHeader_2.54mm:PinHeader_1x02_P2.54mm_Vertical, symbol Connector_Generic:Conn_01x02
- removed PS1: IA0505S, Converter_DCDC:Converter_DCDC_XP_POWER-IAxxxxS_THT, symbol Converter_DCDC:IA0505S
- removed R15, R16, R19: 10E, Resistor_SMD:R_0805_2012Metric_Pad1.20x1.40mm_HandSolder, symbol Device:R_Small
- added C17, C20: 100n, symbol Device:C
- added C18: 1000u, symbol Device:C_Polarized
- added C19: 100u, symbol Device:C_Polarized
- added D4, D5, D6, D7: D, symbol Device:D
- added T1: Transformer_1P_1S, symbol Device:Transformer_1P_1S
- added U4: LM7805_TO220, Package_TO_SOT_THT:TO-220-3_Vertical, symbol Regulator_Linear:LM7805_TO220
- R14, R17, R18, R20, R21, R22: footprint Resistor_SMD:R_0805_2012Metric_Pad1.20x1.40mm_HandSolder -> Resistor_SMD:R_1206_3216Metric_Pad1.30x1.75mm_HandSolder
- R6, R7: value 50m -> 100m
- U1: footprint MCP3911A0-E-SS:MCP3911A0-E&slash_SS -> Package_SO:SSOP-20_5.3x7.2mm_P0.65mm
Connections:
- net SDN is gone; now on net PA5: J7.5 (Pin_5)
- net nIRQ is gone; now on net PA7: J8.1 (Pin_1)
- net +3.3V: now also C16.1, U2.1 (VDD1), U2.7 (EN1)
- net GNDD: no longer D3.1 (K), J6.7 (Pin_7), J9.2 (Pin_2)
- net HIGH_in: now also T1.1 (AA)
- net LOW_in: now also T1.2 (AB)
- net PA5: now also U2.3 (A1)
- net RXD/PA2: now also U2.6 (A4); no longer R17.1, U1.19 (SDO)
- net SCLK: now also U2.4 (A2)
- net SDI: now also U2.5 (A3); no longer R21.1, U1.20 (SDI)
- net GND: now reaches C16.2, U2.2 (GND1), U2.8 (GND1)
- net GND: now also D3.1 (K), J6.7 (Pin_7), J9.2 (Pin_2), C17.2, C18.2, C19.2, C20.2, D6.2 (A), D7.2 (A), U4.2 (GND)
- net LM317_Vin: no longer names the net of C13.1, D2.1 (K), U3.3 (VI)
- net SCK renamed SCK_MCP
- net SCK_: no longer names the net of R18.2, U2.13 (B2)
- net SDI_: no longer names the net of R21.2, U2.12 (B3)
- net SDO_: no longer names the net of R17.2, U2.11 (B4)
- net ~{CS} renamed ~{CS}_MCP
- net ~{CS}_: no longer names the net of R22.2, U2.14 (B1)
- net ~{DR} renamed ~{DR}_MCP
- new net: D4.2 (A), D7.1 (K), T1.4 (SB)
- new net: C17.1, C18.1, D4.1 (K), D5.1 (K), U4.1 (VI)
- new net: D5.2 (A), D6.1 (K), T1.3 (SA)
- new net 5V: C19.1, C20.1, U4.3 (VO)
- new net SDI_MCP: R21.1, U1.20 (SDI)
- new net SDO_MCP: R17.1, U1.19 (SDO)
Other:
- note added: "5V / 1A Netzteil für den Funkchip"
- note removed: "Galvanically isolated voltage output for powering other parts of the module."
- note removed: "MCP3911 IO Ports"
- moved on the sheet: C1, C10, C11, C12, C13, C14, C15, C16, C2, C3, C4, C5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

Commit message: rgergerg
Parts:
- D4, D5, D6, D7: footprint (none) -> Diode_SMD:D_SMA-SMB_Universal_Handsoldering
Other:
- moved on the sheet: C1, C17, C18, C19, C2, C20, C3, C4, C5, C6, D4, D5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

Commit message: power measurement final almost completed
Parts:
- removed C10: 820n/530, Capacitor_THT:C_Rect_L26.5mm_W10.5mm_P22.50mm_MKS4, symbol Power-Analyzer-rescue:C_Small
- removed C17: 100n, symbol Device:C
- removed C19: 100u, symbol Device:C_Polarized
- removed D1: BZG03C15G, Diode_SMD:D_SMA-SMB_Universal_Handsoldering, symbol Power-Analyzer-rescue:D_Zener_Small_ALT
- removed D2: MRA4005T3G, Diode_SMD:D_MicroMELF_Handsoldering, symbol Power-Analyzer-rescue:D_Small
- removed D4, D5, D6, D7: D, Diode_SMD:D_SMA-SMB_Universal_Handsoldering, symbol Device:D
- removed L4: 150n/300m, Inductor_SMD:L_1206_3216Metric, symbol Power-Analyzer-rescue:L_Small
- removed R23: 100E, Resistor_SMD:R_1206_3216Metric_Pad1.30x1.75mm_HandSolder, symbol Power-Analyzer-rescue:R_Small
- removed R24: 1k5, Resistor_SMD:R_1206_3216Metric_Pad1.30x1.75mm_HandSolder, symbol Power-Analyzer-rescue:R_Small
- removed R25: 910, Resistor_SMD:R_1206_3216Metric_Pad1.30x1.75mm_HandSolder, symbol Power-Analyzer-rescue:R_Small
- removed T1: Transformer_1P_1S, symbol Device:Transformer_1P_1S
- removed U4: LM7805_TO220, Package_TO_SOT_THT:TO-220-3_Vertical, symbol Regulator_Linear:LM7805_TO220
- added C17: 6u8, Capacitor_THT:CP_Radial_D10.0mm_P5.00mm, symbol Device:C_Polarized
- added C19: 1n, Capacitor_THT:C_Disc_D11.0mm_W5.0mm_P7.50mm, symbol Device:C
- added C21: 1u, Capacitor_SMD:C_1206_3216Metric_Pad1.33x1.80mm_HandSolder, symbol Device:C_Polarized
- added C22: 1u, Capacitor_SMD:C_1206_3216Metric_Pad1.33x1.80mm_HandSolder, symbol Device:C
- added C23: 1000u, Capacitor_THT:CP_Radial_D10.0mm_P5.00mm, symbol Device:C_Polarized
- added C24: 470u, Capacitor_THT:CP_Radial_D6.3mm_P2.50mm, symbol Device:C_Polarized
- added D10: 1N5822, Diode_THT:D_DO-201AD_P15.24mm_Horizontal, symbol Diode:1N5822
- added D4, D5, D6, D7: 1N4007, Diode_THT:D_DO-41_SOD81_P10.16mm_Horizontal, symbol Diode:1N4007
- added D8: D, Diode_THT:D_DO-201AD_P15.24mm_Horizontal, symbol Device:D
- added D9: 1N4148, Diode_THT:D_DO-35_SOD27_P7.62mm_Horizontal, symbol Diode:1N4148
- added L6, L7: 1m, Inductor_SMD:L_1812_4532Metric_Pad1.30x3.40mm_HandSolder, symbol Device:L
- added R18: 330E, Resistor_SMD:R_1206_3216Metric_Pad1.30x1.75mm_HandSolder, symbol Device:R_Small
- added R18: 270k, Resistor_SMD:R_1206_3216Metric_Pad1.30x1.75mm_HandSolder, symbol Device:R_Small
- added R18 (x2): 28.7k, Resistor_SMD:R_1206_3216Metric_Pad1.30x1.75mm_HandSolder, symbol Device:R_Small
- added R18 (x2): 12E, Resistor_SMD:R_1206_3216Metric_Pad1.30x1.75mm_HandSolder, symbol Device:R_Small
- added R18: 4.42k, Resistor_SMD:R_1206_3216Metric_Pad1.30x1.75mm_HandSolder, symbol Device:R_Small
- added R18: 10E, Resistor_SMD:R_2816_7142Metric_Pad3.20x4.45mm_HandSolder, symbol Device:R_Small
- added R18: 820E, Resistor_SMD:R_1206_3216Metric_Pad1.30x1.75mm_HandSolder, symbol Device:R_Small
- added T1: PA0510NL, Transformer_SMD:Pulse_PA2002NL-PA2008NL-PA2009NL, symbol Transformer:PA0510NL
- added U4: LNK625PG, Package_DIP:PowerIntegrations_PDIP-8C, symbol Regulator_Switching:LNK625PG
- C18: value 1000u -> 6u8; footprint (none) -> Capacitor_THT:CP_Radial_D10.0mm_P5.00mm
- C20: value 100n -> 1u; footprint (none) -> Capacitor_SMD:C_1206_3216Metric_Pad1.33x1.80mm_HandSolder
Connections:
- net +5V is gone; now on net 5V: J9.1 (Pin_1)
- net 5V: now also C13.1, U3.3 (VI), C24.1, L7.2, R18.2; no longer C20.1
- net GND: now also C13.2, C14.2, C15.2, C22.2, C23.2, C24.2, D10.2 (A), R18.1; no longer C18.2, C20.2
- net GNDD: no longer C13.2, C14.2, C15.2
- net HIGH_in: now also R18.1
- net LOW_in: now also D5.1 (K), D7.2 (A)
- net at C18.1: now also C17.1, C19.1, D6.1 (K), D7.1 (K), R18.2, T1.1
- new net: C21.1, D9.1 (K), R18.2
- new net: D9.2 (A), R18.1
- new net: C23.1, L7.1, T1.3
- new net: D4.1 (K), D6.2 (A), R18.2
- new net: C18.2, C20.2, C21.2, L6.2, R18.1, T1.5, U4.5 (S), U4.6 (S), U4.7 (S), U4.8 (S)
- new net: C19.2, R18.1, R18.2
- new net: R18.2, R18.2, T1.4
- new net: D10.1 (K), R18.2, T1.6
- new net: D8.2 (A), T1.8, U4.4 (D)
- new net: D8.1 (K), R18.1
- new net: C20.1, R18.1, U4.2 (BP)
- new net: C22.1, R18.1
- new net: C17.2, D4.2 (A), D5.2 (A), L6.1
- new net: R18.1, R18.2, U4.1 (FB)
Other:
- note added: "1%"
- note added: "10V"
- note added: "16V"
- note added: "1kV"
- note added: "25V"
- note added: "400V"
- note added: "50V"
- note added: "Power Supply"
- note removed: "5V / 1A Netzteil für den Funkchip"
- note removed: "Capacitive power supply"
- note removed: "Power output for ADC"
- moved on the sheet: C1, C11, C12, C16, C2, C3, C4, C5, C6, C7, C8, C9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

Commit message: small fixes
Parts:
- added R24: 1k5, Resistor_SMD:R_1206_3216Metric_Pad1.30x1.75mm_HandSolder, symbol Power-Analyzer-rescue:R_Small
- added R25: 910, Resistor_SMD:R_1206_3216Metric_Pad1.30x1.75mm_HandSolder, symbol Power-Analyzer-rescue:R_Small
- added RV1: 725V, symbol Device:Varistor
Connections:
- net +3.3V: now also R25.1
- net GND: now also R24.2
- net GNDD: now also J1.1 (Pin_1), L3.1, R18.1, R6.1, R7.1
- net HIGH_in: now also D4.1 (K), D6.2 (A), RV1.1; no longer R18.1
- net at U3.1 (ADJ): now also R24.1, R25.2
- removed net LOW_in: D5.1 (K), D7.2 (A), J1.1 (Pin_1), L3.1, R6.1, R7.1
- new net: D5.1 (K), D7.2 (A), R18.2, RV1.2
Other:
- moved on the sheet: C14, C15, R18

Commit message: Power measurement final almst ready
Parts:
- removed C13: 470u, Capacitor_THT:CP_Radial_D10.0mm_P5.00mm, symbol Power-Analyzer-rescue:CP_Small
- removed C14: 100n, Capacitor_SMD:C_1206_3216Metric_Pad1.33x1.80mm_HandSolder, symbol Power-Analyzer-rescue:C_Small
- removed C15: 10u, Capacitor_SMD:C_1206_3216Metric_Pad1.33x1.80mm_HandSolder, symbol Power-Analyzer-rescue:CP_Small
- removed C17, C18: 6u8, Capacitor_THT:CP_Radial_D10.0mm_P5.00mm, symbol Device:C_Polarized
- removed C19: 1n, Capacitor_THT:C_Disc_D11.0mm_W5.0mm_P7.50mm, symbol Device:C
- removed C20, C22: 1u, Capacitor_SMD:C_1206_3216Metric_Pad1.33x1.80mm_HandSolder, symbol Device:C
- removed C21: 1u, Capacitor_SMD:C_1206_3216Metric_Pad1.33x1.80mm_HandSolder, symbol Device:C_Polarized
- removed C23: 1000u, Capacitor_THT:CP_Radial_D10.0mm_P5.00mm, symbol Device:C_Polarized
- removed C24: 470u, Capacitor_THT:CP_Radial_D6.3mm_P2.50mm, symbol Device:C_Polarized
- removed D10: 1N5822, Diode_THT:D_DO-201AD_P15.24mm_Horizontal, symbol Diode:1N5822
- removed D3: LED, Diode_SMD:D_1206_3216Metric_Pad1.42x1.75mm_HandSolder, symbol Device:LED
- removed D4, D5, D6, D7: 1N4007, Diode_THT:D_DO-41_SOD81_P10.16mm_Horizontal, symbol Diode:1N4007
- removed D8: D, Diode_THT:D_DO-201AD_P15.24mm_Horizontal, symbol Device:D
- removed D9: 1N4148, Diode_THT:D_DO-35_SOD27_P7.62mm_Horizontal, symbol Diode:1N4148
- removed L6, L7: 1m, Inductor_SMD:L_1812_4532Metric_Pad1.30x3.40mm_HandSolder, symbol Device:L
- removed R18: 330E, Resistor_SMD:R_1206_3216Metric_Pad1.30x1.75mm_HandSolder, symbol Device:R_Small
- removed R18: 270k, Resistor_SMD:R_1206_3216Metric_Pad1.30x1.75mm_HandSolder, symbol Device:R_Small
- removed R18 (x2): 28.7k, Resistor_SMD:R_1206_3216Metric_Pad1.30x1.75mm_HandSolder, symbol Device:R_Small
- removed R18 (x2): 12E, Resistor_SMD:R_1206_3216Metric_Pad1.30x1.75mm_HandSolder, symbol Device:R_Small
- removed R18: 4.42k, Resistor_SMD:R_1206_3216Metric_Pad1.30x1.75mm_HandSolder, symbol Device:R_Small
- removed R18: 10E, Resistor_SMD:R_2816_7142Metric_Pad3.20x4.45mm_HandSolder, symbol Device:R_Small
- removed R18: 820E, Resistor_SMD:R_1206_3216Metric_Pad1.30x1.75mm_HandSolder, symbol Device:R_Small
- removed R24: 1k5, Resistor_SMD:R_1206_3216Metric_Pad1.30x1.75mm_HandSolder, symbol Power-Analyzer-rescue:R_Small
- removed R25: 910, Resistor_SMD:R_1206_3216Metric_Pad1.30x1.75mm_HandSolder, symbol Power-Analyzer-rescue:R_Small
- removed RV1: 725V, symbol Device:Varistor
- removed T1: PA0510NL, Transformer_SMD:Pulse_PA2002NL-PA2008NL-PA2009NL, symbol Transformer:PA0510NL
- removed U3: LM317_TO-252, Package_TO_SOT_SMD:TO-252-2, symbol Regulator_Linear:LM317_TO-252
- removed U4: LNK625PG, Package_DIP:PowerIntegrations_PDIP-8C, symbol Regulator_Switching:LNK625PG
- added C?: 820n/530, Capacitor_THT:C_Rect_L26.5mm_W10.5mm_P22.50mm_MKS4, symbol Power-Analyzer-rescue:C_Small
- added C?: 100n, Capacitor_SMD:C_1206_3216Metric_Pad1.33x1.80mm_HandSolder, symbol Power-Analyzer-rescue:C_Small
- added C?: 10u, Capacitor_SMD:C_1206_3216Metric_Pad1.33x1.80mm_HandSolder, symbol Power-Analyzer-rescue:CP_Small
- added C?: 470u, Capacitor_THT:CP_Radial_D10.0mm_P5.00mm, symbol Power-Analyzer-rescue:CP_Small
- added D?: BZG03C15G, Diode_SMD:D_SMA-SMB_Universal_Handsoldering, symbol Power-Analyzer-rescue:D_Zener_Small_ALT
- added D?: MRA4005T3G, Diode_SMD:D_MicroMELF_Handsoldering, symbol Power-Analyzer-rescue:D_Small
- added J10, J12, J13, J9: Conn_01x01_Pin, Connector_PinHeader_2.54mm:PinHeader_1x01_P2.54mm_Vertical, symbol Connector:Conn_01x01_Pin
- added J11: Conn_01x02_Pin, Connector_PinHeader_2.54mm:PinHeader_1x02_P2.54mm_Vertical, symbol Connector:Conn_01x02_Pin
- added J7: RFShield_OnePiece, RF_Shielding:Laird_Technologies_BMI-S-209-F_29.36x18.50mm, symbol Device:RFShield_OnePiece
- added JP1: cap psu jp, Connector_PinHeader_2.54mm:PinHeader_1x02_P2.54mm_Vertical, symbol Jumper:Jumper_2_Bridged
- added L?: 150n/300m, Inductor_SMD:L_1206_3216Metric, symbol Power-Analyzer-rescue:L_Small
- added R13: 1k, Resistor_SMD:R_1206_3216Metric, symbol Device:R_Small
- added R14: 100k, Resistor_SMD:R_1206_3216Metric, symbol Device:R_Small
- added R?: 1k5, Resistor_SMD:R_1206_3216Metric_Pad1.30x1.75mm_HandSolder, symbol Power-Analyzer-rescue:R_Small
- added R?: 100E, Resistor_SMD:R_1206_3216Metric_Pad1.30x1.75mm_HandSolder, symbol Power-Analyzer-rescue:R_Small
- added R?: 910, Resistor_SMD:R_1206_3216Metric_Pad1.30x1.75mm_HandSolder, symbol Power-Analyzer-rescue:R_Small
- added U3: CNY17-3, Package_DIP:DIP-6_W7.62mm_LongPads, symbol Isolator:CNY17-3
- added U?: LM317_TO-252, Package_TO_SOT_SMD:TO-252-2, symbol Regulator_Linear:LM317_TO-252
- J4: renamed from J5; footprint Connector_PinSocket_2.54mm:PinSocket_1x07_P2.54mm_Vertical -> Connector_PinSocket_2.54mm:PinSocket_1x09_P2.54mm_Vertical; symbol Connector:Conn_01x07_Socket -> Connector:Conn_01x09_Socket
- J5: renamed from J6; footprint Connector_PinSocket_2.54mm:PinSocket_1x07_P2.54mm_Vertical -> Connector_PinSocket_2.54mm:PinSocket_1x09_P2.54mm_Vertical; symbol Connector:Conn_01x07_Socket -> Connector:Conn_01x09_Socket
- J8: renamed from J10; footprint Connector_PinSocket_2.54mm:PinSocket_1x03_P2.54mm_Vertical -> Connector_PinHeader_2.54mm:PinHeader_1x05_P2.54mm_Vertical; symbol Connector:Conn_01x03_Socket -> Connector:Conn_01x05_Pin
- J?: renamed from J1; footprint TerminalBlock:TerminalBlock_Altech_AK300-4_P5.00mm -> Connector_Phoenix_MSTB:PhoenixContact_MSTBVA_2,5_4-G-5,08_1x04_P5.08mm_Vertical
- R?: renamed from R20; footprint Resistor_SMD:R_1206_3216Metric_Pad1.30x1.75mm_HandSolder -> Resistor_SMD:R_0805_2012Metric_Pad1.20x1.40mm_HandSolder
- R?: renamed from R22; footprint Resistor_SMD:R_1206_3216Metric_Pad1.30x1.75mm_HandSolder -> Resistor_SMD:R_0805_2012Metric_Pad1.20x1.40mm_HandSolder
- R?: renamed from R18; footprint Resistor_SMD:R_1206_3216Metric_Pad1.30x1.75mm_HandSolder -> Resistor_SMD:R_0805_2012Metric_Pad1.20x1.40mm_HandSolder
- R?: renamed from R17; footprint Resistor_SMD:R_1206_3216Metric_Pad1.30x1.75mm_HandSolder -> Resistor_SMD:R_0805_2012Metric_Pad1.20x1.40mm_HandSolder
- R?: renamed from R21; footprint Resistor_SMD:R_1206_3216Metric_Pad1.30x1.75mm_HandSolder -> Resistor_SMD:R_0805_2012Metric_Pad1.20x1.40mm_HandSolder
- renumbered C5 to C?, C9 to C?, C16 to C?, C8 to C?, C4 to C?, C2 to C?, C7 to C?, C3 to C?, C6 to C?, C12 to C?, C11 to C?, C1 to C?, FB1 to FB?, J9 to J2, J8 to J3, J7 to J6, L3 to L?, L1 to L?, L2 to L?, L5 to L?, R26 to R25, R8 to R?, R10 to R?, R13 to R?, R5 to R?, R14 to R?, R11 to R?, R3 to R?, R12 to R?, R9 to R?, R2 to R?, R1 to R?, R6 to R?, R7 to R?, R4 to R?, U2 to U?, U1 to U?, Y1 to Y?
Connections:
- net +3.3V: now also C?.1, C?.1, R?.1, U?.2 (VO); no longer C?.1, J4.1 (Pin_1), U?.1 (VDD1), U?.7 (EN1)
- net 3V3D: now also R13.2, R14.1
- net CH0+: now also C?.1, R?.2; no longer C?.2, R?.2
- net CH0-: now also C?.2, R?.2; no longer C?.1, R?.2
- net CH1+: now also C?.1, R?.2, U?.7 (CH1+); no longer C?.1, R?.2, U?.6 (CH1-)
- net CH1-: now also C?.2, R?.2, U?.6 (CH1-); no longer C?.2, R?.2, U?.7 (CH1+)
- net GND: now also J5.1 (Pin_1), J8.1 (Pin_1), J10.1 (Pin_1), J11.1 (Pin_1), U3.2; no longer J5.7 (Pin_7)
- net GNDA: now also J7.1 (Shield)
- net GNDD: now also C?.2, C?.2, C?.2, D?.2 (A), J9.1 (Pin_1), R?.2, U3.4
- net GPIO0: now also J4.8 (Pin_8)
- net GPIO1: now also J4.9 (Pin_9)
- net HIGH_in: now also JP1.1 (A)
- net PA6: now also J6.5 (Pin_5); no longer J6.1 (Pin_1)
- net RESET-UDPI: now also J5.5 (Pin_5), J8.5 (Pin_5); no longer J5.3 (Pin_3), J8.1 (Pin_1)
- net RxD/PB3: now also J8.4 (Pin_4); no longer J8.2 (Pin_2)
- net SCL/XDIR/PB0: now also J5.6 (Pin_6), U3.1; no longer J5.2 (Pin_2)
- net SDA/XCK/PB1: now also J5.7 (Pin_7), R25.1; no longer J5.1 (Pin_1)
- net ~{DR}_MCP: now also R14.2
- net ~{RESET}: now also U3.6
- net at R25.2: now also J11.2 (Pin_2)
- net 5V renamed +5V
- net +5V: now also C?.1, J4.1 (Pin_1), J8.2 (Pin_2), U?.1 (VDD1), U?.7 (EN1), J13.1 (Pin_1)
- removed net PA5: J4.3 (Pin_3), J6.5 (Pin_5), R25.1, U?.3 (A1)
- net RXD/PA2 renamed MISO
- net MISO: now also J5.3 (Pin_3); no longer J5.5 (Pin_5)
- net SCLK renamed SCK
- net SCK: now also J5.2 (Pin_2); no longer J5.6 (Pin_6)
- net SDI renamed MOSI
- net XDIR/PA4 renamed CS_adc
- net CS_adc: now also U?.3 (A1)
- new net: R13.1, U3.5
- new net: R?.1, R?.2, U?.1 (ADJ)
- new net: JP1.2 (B), L?.1
- new net: C?.1, L?.2
- new net: D?.1 (K), D?.2 (A), R?.2
- new net CS_funk: J4.3 (Pin_3), J6.1 (Pin_1)
- new net LM317_input: C?.1, D?.1 (K), J12.1 (Pin_1), U?.3 (VI)
- new net x_cap_out: C?.2, R?.1
- no-connect marks 6 -> 8
Other:
- note added: "Capacitive power supply - Power Measurement - Side"
- note added: "Power output for ADC"
- note removed: "1%"
- note removed: "10V"
- note removed: "16V"
- note removed: "1kV"
- note removed: "25V"
- note removed: "400V"
- note removed: "50V"
- note removed: "Power Supply"
- moved on the sheet: C?, J2, J3, J6, L?, R25, R?, U?

Commit message: various fixes
Parts:
- added D3, D4: D_Schottky, symbol Device:D_Schottky
- added R?: 10E, Resistor_SMD:R_0805_2012Metric_Pad1.20x1.40mm_HandSolder, symbol Device:R_Small
- J5: footprint Connector_PinSocket_2.54mm:PinSocket_1x09_P2.54mm_Vertical -> Connector_PinSocket_2.54mm:PinSocket_1x07_P2.54mm_Vertical
- R?: footprint Resistor_SMD:R_1206_3216Metric_Pad1.30x1.75mm_HandSolder -> Resistor_SMD:R_0805_2012Metric_Pad1.20x1.40mm_HandSolder
Connections:
- net ~{RESET}: now also R?.1; no longer U3.6
- new net: R?.2, U3.6
Other:
- moved on the sheet: J10, J12, J13, J9
