File: power-measurement-final/power-measurement-final/power-measurement-final.kicad_pcb (KiCad board)
At the start: 4 copper layers, 89 x 89 mm, 62 parts, among them J1 Screw_Terminal_01x04, J2 Conn_01x09, J3 Conn_01x07, J4 Conn_01x02, J5 Conn_01x07_Socket, J6 Conn_01x07_Socket, J7 Conn_01x05_Socket, J8 Conn_01x03_Socket, J9 Conn_01x02_Socket, U2 Si8641BA-B-IU, U3 LM317_TO-252, Y1 10M

Commit message: power measuremnt final weitergemacht
Parts:
- added D3: LED, Diode_SMD:D_1206_3216Metric_Pad1.42x1.75mm_HandSolder, F.Cu at (176.0, 116.1)
- added J10: Conn_01x03_Socket, Connector_PinSocket_2.54mm:PinSocket_1x03_P2.54mm_Vertical, F.Cu at (166.9, 141.5)
- added R26: 330, Resistor_SMD:R_1206_3216Metric_Pad1.30x1.75mm_HandSolder, F.Cu at (177.5, 122.3)
- added TP1: TestPoint, TestPoint:TestPoint_Plated_Hole_D3.0mm, F.Cu at (183.0, 60.9)
- added TP2: TestPoint, TestPoint:TestPoint_Plated_Hole_D3.0mm, F.Cu at (100.0, 61.1)
- added TP3: TestPoint, TestPoint:TestPoint_Plated_Hole_D3.0mm, F.Cu at (182.8, 143.7)
- added TP4: TestPoint, TestPoint:TestPoint_Plated_Hole_D3.0mm, F.Cu at (100.3, 143.7)
- moved R15 103.2 mm to (237.9, 119.7)
- moved R16 103.2 mm to (237.9, 122.6)
- moved R17 103.2 mm to (237.9, 125.6)
- moved R18 103.2 mm to (237.9, 128.5)
- moved R19 103.2 mm to (237.9, 131.5)
- moved R22 103.2 mm to (237.9, 140.3)
- moved R21 103.2 mm to (237.9, 137.4)
- moved C12 81.4 mm to (229.5, 90.1)
- moved C16 81.4 mm to (229.5, 100.2)
- moved J2 81.4 mm to (209.0, 110.9)
- moved U2 81.4 mm to (227.0, 115.1)
- moved J3 81.4 mm to (221.3, 124.9)
- moved J4 52.9 mm to (121.0, 72.5), turned to 180 degrees
- moved J5 43.6 mm to (182.5, 136.7)
- moved J6 43.6 mm to (167.1, 121.5)
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Connections:
- net /Antenne renamed +5V
- J6 pad 4: /TXD/PA1 -> /SDI
- J6 pad 6: /XCK/PA3 -> /SCLK
- J7 pad 1: /nSEL -> /PA6
- J7 pad 2: /SDO -> /RXD/PA2
- J9 pad 2: unconnected-(J9-Pin_2-Pad2) -> GNDD
- R17 pad 1: /SDO -> /RXD/PA2
Routing:
- net +3.3V: track 116.3 -> 176.0 mm, vias 0 -> 2
- net /PA6: track 0.23 -> 37.8 mm
- net /TxD/PB2: track 0.00 -> 26.0 mm
- net /RxD/PB3: track 0.00 -> 23.5 mm
- net /RESET-UDPI: track 0.04 -> 17.9 mm
- net /PA5: track 0.00 -> 14.8 mm, vias 0 -> 1
- net /RXD/PA2: track 0.00 -> 14.2 mm
- net /SDI: track 0.57 -> 10.1 mm
- net /5V_ext: track 0.00 -> 9.35 mm
- net /GND_ext: track 0.00 -> 9.35 mm
- net /SCLK: track 0.00 -> 8.62 mm
- net Net-(L1-Pad2): track 14.9 -> 22.9 mm
- net Net-(L3-Pad2): track 3.71 -> 10.5 mm
- net /voltage_pos: track 25.7 -> 20.9 mm
- net Net-(R5-Pad2): track 26.3 -> 21.6 mm
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- added copper zone on In1.Cu, net (none)
- added copper zone on In2.Cu, net (none)
- added copper zone on B.Cu, net GNDA
- added copper zone on F.Cu, net GNDD
Other:
- outline, holes or cut-outs redrawn
- board text added: "ATtiny status led"
- board text added: "RxD"
- board text added: "TxD"
- board text added: "UDPI"

Commit message: finales power measurement modul weitergemacht
Parts:
- removed J2: Conn_01x09, Connector_PinHeader_2.54mm:PinHeader_1x09_P2.54mm_Vertical
- removed J3: Conn_01x07, Connector_PinHeader_2.54mm:PinHeader_1x07_P2.54mm_Vertical
- removed J4: Conn_01x02, Connector_PinHeader_2.54mm:PinHeader_1x02_P2.54mm_Vertical
- removed PS1: IA0505S, Converter_DCDC:Converter_DCDC_XP_POWER-IAxxxxS_THT
- removed R15, R16, R19: 10E, Resistor_SMD:R_0805_2012Metric_Pad1.20x1.40mm_HandSolder
- added U1: MCP3911A0-E-SS, Package_SO:SSOP-20_5.3x7.2mm_P0.65mm, B.Cu at (129.0, 108.7)
- C12, C16, U2: moved to B.Cu
- R14, R20: footprint Resistor_SMD:R_0805_2012Metric_Pad1.20x1.40mm_HandSolder -> Resistor_SMD:R_1206_3216Metric_Pad1.30x1.75mm_HandSolder
- R17, R18, R21, R22: footprint Resistor_SMD:R_0805_2012Metric_Pad1.20x1.40mm_HandSolder -> Resistor_SMD:R_1206_3216Metric_Pad1.30x1.75mm_HandSolder; moved to B.Cu
- R6, R7: value 50m -> 100m
- moved C12 127.7 mm to (106.4, 124.1), turned to -90 degrees
- moved C16 114.3 mm to (118.2, 126.4), turned to 90 degrees
- moved R17 106.4 mm to (131.6, 123.8), turned to -90 degrees
- moved R18 103.5 mm to (134.5, 123.8), turned to -90 degrees
- moved U2 102.2 mm to (126.7, 134.5)
- moved R21 101.2 mm to (137.7, 123.8), turned to -90 degrees
- moved R22 98.7 mm to (140.6, 123.8), turned to -90 degrees
- moved D3 5.90 mm to (181.9, 116.2)
- moved C4 2.94 mm to (136.4, 64.1)
- moved C5 2.94 mm to (136.4, 67.4)
- moved C3 2.94 mm to (136.2, 60.7)
- moved R10 2.94 mm to (142.7, 60.9)
- moved R11 2.94 mm to (142.7, 64.2)
- moved R12 2.94 mm to (142.7, 67.5)
- moved R9 2.94 mm to (147.2, 62.1)
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Connections:
- net /LM317_Vin renamed Net-(D2-K)
- net /SCK_ renamed Net-(U2-B2)
- net /SDI_ renamed Net-(U2-B3)
- net /SDO_ renamed Net-(U2-B4)
- net /~{CS}_ renamed Net-(U2-B1)
- C16 pad 1: Net-(J3-Pin_1) -> +3.3V
- C16 pad 2: Net-(J3-Pin_2) -> GND
- D3 pad 1: GNDD -> GND
- J6 pad 7: GNDD -> GND
- J7 pad 5: /SDN -> /PA5
- J8 pad 1: /nIRQ -> /PA7
- J9 pad 2: GNDD -> GND
- R17 pad 1: /RXD/PA2 -> /SDO_MCP
- R18 pad 1: /SCK -> /SCK_MCP
- R21 pad 1: /SDI -> /SDI_MCP
- R22 pad 1: /~{CS} -> /~{CS}_MCP
- U2 pad 1: Net-(J3-Pin_1) -> +3.3V
- U2 pad 2: Net-(J3-Pin_2) -> GND
- U2 pad 3: Net-(J3-Pin_3) -> /PA5
- U2 pad 4: Net-(J3-Pin_4) -> /SCLK
- U2 pad 5: Net-(J3-Pin_5) -> /SDI
- U2 pad 6: Net-(J3-Pin_6) -> /RXD/PA2
- U2 pad 7: Net-(J3-Pin_7) -> +3.3V
- U2 pad 8: Net-(J3-Pin_2) -> GND
Routing:
- net GND: track 0.00 -> 106.0 mm, vias 0 -> 1
- net /PA5: track 14.8 -> 96.1 mm
- net /3V3D: track 3.22 -> 76.8 mm
- net /CH0-: track 4.87 -> 64.7 mm, vias 0 -> 2
- net /CH0+: track 30.2 -> 81.1 mm, vias 0 -> 2
- net /CH1+: track 3.20 -> 53.0 mm, vias 0 -> 2
- net /PA7: track 0.00 -> 45.8 mm, vias 0 -> 2
- net /SCLK: track 8.62 -> 50.8 mm, vias 0 -> 1
- net /RXD/PA2: track 14.2 -> 56.1 mm, vias 0 -> 1
- net /SDI: track 10.1 -> 51.7 mm, vias 0 -> 1
- net /CH1-: track 7.46 -> 47.7 mm, vias 0 -> 2
- net /OSC1: track 9.67 -> 37.2 mm, vias 0 -> 2
- net /3V3A: track 3.01 -> 28.9 mm, vias 0 -> 2
- net /OSC2: track 9.44 -> 34.9 mm, vias 0 -> 2
- net +3.3V: track 176.0 -> 201.1 mm, vias 2 -> 4
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- removed copper zone on B.Cu, net GNDA
Other:
- outline, holes or cut-outs redrawn

Commit message: rgergerg
Parts:
- moved C16 34.1 mm to (147.0, 144.7), turned to 180 degrees
- moved U2 23.4 mm to (149.9, 131.0)
- moved Y1 22.3 mm to (113.6, 79.0)
- moved C2 22.2 mm to (118.7, 85.7)
- moved R1 21.6 mm to (118.7, 81.4)
- moved C1 21.1 mm to (118.7, 77.0)
- moved C12 20.9 mm to (110.7, 103.6), turned to 0 degrees
- moved R17 19.8 mm to (151.2, 121.4), turned to 0 degrees
- moved R18 17.6 mm to (151.2, 118.5), turned to 0 degrees
- moved C13 17.4 mm to (115.0, 69.3)
- moved R21 16.0 mm to (151.2, 115.3), turned to 0 degrees
- moved R22 15.6 mm to (151.2, 112.3), turned to 0 degrees
- moved C11 15.1 mm to (106.2, 103.3)
- moved FB1 15.1 mm to (100.9, 99.7)
- moved L5 15.1 mm to (109.4, 99.1)
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Routing:
- net /PA5: track 96.1 -> 72.4 mm, vias 1 -> 3
- net /3V3D: track 76.8 -> 55.6 mm, vias 0 -> 1
- net +3.3V: track 201.1 -> 183.4 mm, vias 4 -> 5
- net /SDI_MCP: track 21.9 -> 38.2 mm
- net /OSC1: track 37.2 -> 53.0 mm
- net /SDO_MCP: track 12.0 -> 27.6 mm
- net /RXD/PA2: track 56.1 -> 42.2 mm, vias 1 -> 2
- net GND: track 106.0 -> 119.2 mm, vias 1 -> 5
- net /SCK_MCP: track 13.0 -> 25.9 mm
- net /SCLK: track 50.8 -> 38.1 mm, vias 1 -> 2
- net /OSC2: track 34.9 -> 46.5 mm
- net /SDI: track 51.7 -> 42.9 mm, vias 1 -> 0
- net GNDA: track 109.9 -> 101.7 mm
- net /~{CS}_MCP: track 17.3 -> 23.7 mm
- net Net-(U2-B1): track 18.1 -> 23.9 mm
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
Commit message: power measurement final almost completed
Parts:
- removed C10: 820n/530, Capacitor_THT:C_Rect_L26.5mm_W10.5mm_P22.50mm_MKS4
- removed C13: 470u, Capacitor_THT:CP_Radial_D10.0mm_P5.00mm
- removed C14: 100n, Capacitor_SMD:C_1206_3216Metric_Pad1.33x1.80mm_HandSolder
- removed C15: 10u, Capacitor_SMD:C_1206_3216Metric_Pad1.33x1.80mm_HandSolder
- removed D1: BZG03C15G, Diode_SMD:D_SMA-SMB_Universal_Handsoldering
- removed D2: MRA4005T3G, Diode_SMD:D_MicroMELF_Handsoldering
- removed L4: 150n/300m, Inductor_SMD:L_1206_3216Metric
- removed R23: 100E, Resistor_SMD:R_1206_3216Metric_Pad1.30x1.75mm_HandSolder
- removed R24: 1k5, Resistor_SMD:R_1206_3216Metric_Pad1.30x1.75mm_HandSolder
- removed R25: 910, Resistor_SMD:R_1206_3216Metric_Pad1.30x1.75mm_HandSolder
- removed U3: LM317_TO-252, Package_TO_SOT_SMD:TO-252-2
- added C17: 6u8, Capacitor_THT:CP_Radial_D10.0mm_P5.00mm, F.Cu at (121.8, 66.4)
- added C18: 6u8, Capacitor_THT:CP_Radial_D10.0mm_P5.00mm, F.Cu at (109.8, 61.6)
- added C19: 1n, Capacitor_THT:C_Disc_D11.0mm_W5.0mm_P7.50mm, F.Cu at (101.0, 67.5)
- added C20: 1u, Capacitor_SMD:C_1206_3216Metric_Pad1.33x1.80mm_HandSolder, B.Cu at (129.9, 83.4)
- added C21: 1u, Capacitor_SMD:C_1206_3216Metric_Pad1.33x1.80mm_HandSolder, B.Cu at (134.8, 88.2)
- added C22: 1u, Capacitor_SMD:C_1206_3216Metric_Pad1.33x1.80mm_HandSolder, B.Cu at (102.2, 85.0)
- added C23: 1000u, Capacitor_THT:CP_Radial_D10.0mm_P5.00mm, F.Cu at (110.3, 89.5)
- added C24: 470u, Capacitor_THT:CP_Radial_D6.3mm_P2.50mm, F.Cu at (118.3, 90.7)
- added C25: 470u, Capacitor_THT:CP_Radial_D10.0mm_P5.00mm, F.Cu at (126.2, 94.0)
- added C26: 100n, Capacitor_SMD:C_1206_3216Metric_Pad1.33x1.80mm_HandSolder, B.Cu at (128.8, 89.8)
- added C27: 10u, Capacitor_SMD:C_1206_3216Metric_Pad1.33x1.80mm_HandSolder, B.Cu at (125.5, 89.8)
- added D10: 1N5822, Diode_THT:D_DO-201AD_P15.24mm_Horizontal, F.Cu at (101.0, 79.8)
- added D4: 1N4007, Diode_THT:D_DO-41_SOD81_P10.16mm_Horizontal, F.Cu at (129.9, 70.2)
- added D5: 1N4007, Diode_THT:D_DO-41_SOD81_P10.16mm_Horizontal, F.Cu at (134.3, 70.2)
- added D6: 1N4007, Diode_THT:D_DO-41_SOD81_P10.16mm_Horizontal, F.Cu at (143.1, 59.9)
- added D7: 1N4007, Diode_THT:D_DO-41_SOD81_P10.16mm_Horizontal, F.Cu at (138.5, 59.9)
- added D8: D, Diode_THT:D_DO-201AD_P15.24mm_Horizontal, F.Cu at (110.6, 73.0)
- added D9: 1N4148, Diode_THT:D_DO-35_SOD27_P7.62mm_Horizontal, F.Cu at (139.7, 88.2)
- added L6: 1m, Inductor_SMD:L_1812_4532Metric_Pad1.30x3.40mm_HandSolder, B.Cu at (117.1, 66.4)
- added L7: 1m, Inductor_SMD:L_1812_4532Metric_Pad1.30x3.40mm_HandSolder, B.Cu at (105.2, 90.2)
- added R15: 10E, Resistor_SMD:R_2816_7142Metric_Pad3.20x4.45mm_HandSolder, B.Cu at (155.5, 92.8)
- added R16: 270k, Resistor_SMD:R_1206_3216Metric_Pad1.30x1.75mm_HandSolder, B.Cu at (103.5, 71.2)
- added R19: 330E, Resistor_SMD:R_1206_3216Metric_Pad1.30x1.75mm_HandSolder, B.Cu at (106.6, 71.2)
- added R27: 28.7k, Resistor_SMD:R_1206_3216Metric_Pad1.30x1.75mm_HandSolder, B.Cu at (131.0, 77.5)
- added R28: 4.42k, Resistor_SMD:R_1206_3216Metric_Pad1.30x1.75mm_HandSolder, B.Cu at (133.1, 83.3)
- added R29: 12E, Resistor_SMD:R_1206_3216Metric_Pad1.30x1.75mm_HandSolder, B.Cu at (136.5, 77.5)
- added R30: 28.7k, Resistor_SMD:R_1206_3216Metric_Pad1.30x1.75mm_HandSolder, B.Cu at (136.3, 83.3)
- added R31: 12E, Resistor_SMD:R_1206_3216Metric_Pad1.30x1.75mm_HandSolder, B.Cu at (99.4, 85.0)
- added R32: 820E, Resistor_SMD:R_1206_3216Metric_Pad1.30x1.75mm_HandSolder, B.Cu at (116.6, 88.2)
- added T1: PA0510NL, Transformer_SMD:Pulse_PA2002NL-PA2008NL-PA2009NL, B.Cu at (109.0, 81.4)
- added U4: LNK625PG, Package_DIP:PowerIntegrations_PDIP-8C, F.Cu at (126.1, 77.6)
- added U5: LM317_TO-252, Package_TO_SOT_SMD:TO-252-2, B.Cu at (117.8, 96.0)
- moved Y1 64.4 mm to (107.5, 143.1), turned to 0 degrees
- moved C16 63.0 mm to (105.0, 97.7), turned to 90 degrees
- moved C1 59.8 mm to (100.2, 133.9), turned to 90 degrees
- moved R1 58.7 mm to (101.7, 137.6), turned to 0 degrees
- moved R11 56.7 mm to (107.7, 108.9)
- moved C4 56.7 mm to (101.4, 108.8)
- moved R10 56.7 mm to (107.7, 105.6)
- moved R12 56.7 mm to (107.7, 112.2)
- moved R13 56.7 mm to (107.7, 115.5)
- moved C3 56.7 mm to (101.2, 105.4)
- moved R9 56.7 mm to (112.2, 106.8)
- moved C5 56.7 mm to (101.7, 112.3)
- moved C6 56.3 mm to (101.8, 116.0)
- moved C2 50.7 mm to (103.2, 134.0), turned to 90 degrees
- moved R3 45.9 mm to (110.1, 119.8), turned to 90 degrees
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Connections:
- net HIGH_in renamed /HIGH_in
- J9 pad 1: +5V -> /5V
Routing:
- net GND: track 119.2 -> 27.6 mm, vias 5 -> 1
- net GNDA: track 101.7 -> 20.5 mm, vias 5 -> 0
- net Net-(D6-K): track 0.00 -> 74.5 mm
- net Net-(L3-Pad2): track 11.1 -> 82.6 mm, vias 0 -> 2
- net /5V: track 0.00 -> 71.0 mm, vias 0 -> 2
- net Net-(C10-Pad1): track 69.0 -> 0.00 mm
- net Net-(L2-Pad2): track 8.89 -> 77.8 mm, vias 0 -> 2
- net Net-(C18-Pad2): track 0.00 -> 56.4 mm
- net +3.3V: track 183.4 -> 134.6 mm, vias 5 -> 2
- net /x_cap_out: track 47.3 -> 0.00 mm
- net Net-(L1-Pad2): track 22.9 -> 69.3 mm, vias 0 -> 2
- net Net-(D4-K): track 0.00 -> 43.6 mm
- net /CH0-: track 64.5 -> 23.1 mm
- net Net-(D1-K): track 35.7 -> 0.00 mm, vias 3 -> 0
- net /CH0+: track 81.1 -> 47.0 mm, vias 2 -> 0
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- added copper zone on B.Cu, net GND
- added copper zone on F.Cu, net GND
- added copper zone on In1.Cu, net GND
- added copper zone on In2.Cu, net GND
- added copper zone on B.Cu, net GNDA
- removed copper zone on F.Cu, net GNDD
Other:
- outline, holes or cut-outs redrawn

Commit message: Power measurement final almst ready
Parts:
- removed C17, C18: 6u8, Capacitor_THT:CP_Radial_D10.0mm_P5.00mm
- removed C19: 1n, Capacitor_THT:C_Disc_D11.0mm_W5.0mm_P7.50mm
- removed C20, C21, C22: 1u, Capacitor_SMD:C_1206_3216Metric_Pad1.33x1.80mm_HandSolder
- removed C23: 1000u, Capacitor_THT:CP_Radial_D10.0mm_P5.00mm
- removed C24: 470u, Capacitor_THT:CP_Radial_D6.3mm_P2.50mm
- removed C25: 470u, Capacitor_THT:CP_Radial_D10.0mm_P5.00mm
- removed C26: 100n, Capacitor_SMD:C_1206_3216Metric_Pad1.33x1.80mm_HandSolder
- removed C27: 10u, Capacitor_SMD:C_1206_3216Metric_Pad1.33x1.80mm_HandSolder
- removed D10: 1N5822, Diode_THT:D_DO-201AD_P15.24mm_Horizontal
- removed D3: LED, Diode_SMD:D_1206_3216Metric_Pad1.42x1.75mm_HandSolder
- removed D4, D5, D6, D7: 1N4007, Diode_THT:D_DO-41_SOD81_P10.16mm_Horizontal
- removed D8: D, Diode_THT:D_DO-201AD_P15.24mm_Horizontal
- removed D9: 1N4148, Diode_THT:D_DO-35_SOD27_P7.62mm_Horizontal
- removed the L5 at (106.3, 129.1)
- removed L6, L7: 1m, Inductor_SMD:L_1812_4532Metric_Pad1.30x3.40mm_HandSolder
- removed the R20 at (100.3, 129.2)
- removed R27, R30: 28.7k, Resistor_SMD:R_1206_3216Metric_Pad1.30x1.75mm_HandSolder
- removed R28: 4.42k, Resistor_SMD:R_1206_3216Metric_Pad1.30x1.75mm_HandSolder
- removed R29, R31: 12E, Resistor_SMD:R_1206_3216Metric_Pad1.30x1.75mm_HandSolder
- removed R32: 820E, Resistor_SMD:R_1206_3216Metric_Pad1.30x1.75mm_HandSolder
- removed the R4 at (113.5, 115.4)
- removed the R5 at (113.5, 112.1)
- removed T1: PA0510NL, Transformer_SMD:Pulse_PA2002NL-PA2008NL-PA2009NL
- removed U5: LM317_TO-252, Package_TO_SOT_SMD:TO-252-2
- added C10: 100n, Capacitor_SMD:C_1206_3216Metric_Pad1.33x1.80mm_HandSolder, B.Cu at (142.0, 108.0)
- added C13: 820n/530, Capacitor_THT:C_Rect_L26.5mm_W10.5mm_P22.50mm_MKS4, F.Cu at (155.8, 63.5)
- added C14: 470u, Capacitor_THT:CP_Radial_D10.0mm_P5.00mm, F.Cu at (114.4, 66.3)
- added C15: 100n, Capacitor_SMD:C_1206_3216Metric_Pad1.33x1.80mm_HandSolder, B.Cu at (112.5, 85.6)
- added D1: BZG03C15G, Diode_SMD:D_SMA-SMB_Universal_Handsoldering, B.Cu at (121.8, 65.7)
- added D2: MRA4005T3G, Diode_SMD:D_MicroMELF_Handsoldering, B.Cu at (121.9, 69.1)
- added J10: Conn_01x01_Pin, Connector_PinHeader_2.54mm:PinHeader_1x01_P2.54mm_Vertical, F.Cu at (110.5, 100.1)
- added J11: Conn_01x02_Pin, Connector_PinHeader_2.54mm:PinHeader_1x02_P2.54mm_Vertical, F.Cu at (176.8, 110.5)
- added J12: Conn_01x01_Pin, Connector_PinHeader_2.54mm:PinHeader_1x01_P2.54mm_Vertical, F.Cu at (120.4, 72.1)
- added J13: Conn_01x01_Pin, Connector_PinHeader_2.54mm:PinHeader_1x01_P2.54mm_Vertical, F.Cu at (108.2, 96.0)
- added J7: RFShield_OnePiece, RF_Shielding:Laird_Technologies_BMI-S-209-F_29.36x18.50mm, B.Cu at (139.4, 81.6)
- added J9: Conn_01x01_Pin, Connector_PinHeader_2.54mm:PinHeader_1x01_P2.54mm_Vertical, F.Cu at (117.9, 90.4)
- added JP1: cap psu jp, Connector_PinHeader_2.54mm:PinHeader_1x02_P2.54mm_Vertical, F.Cu at (166.4, 61.5)
- added L1: 150n/300m, Inductor_SMD:L_1206_3216Metric, B.Cu at (131.2, 86.9)
- added L4: 150n/300m, Inductor_SMD:L_1206_3216Metric, B.Cu at (160.5, 64.8)
- added R17: 100E, Resistor_SMD:R_1206_3216Metric_Pad1.30x1.75mm_HandSolder, B.Cu at (129.3, 64.6)
- added R18: 180k, Resistor_SMD:R_1206_3216Metric_Pad1.30x1.75mm_HandSolder, B.Cu at (161.2, 94.2)
- added R23: 1k5, Resistor_SMD:R_1206_3216Metric_Pad1.30x1.75mm_HandSolder, B.Cu at (110.4, 71.4)
- added R24: 910, Resistor_SMD:R_1206_3216Metric_Pad1.30x1.75mm_HandSolder, B.Cu at (115.7, 75.1)
- added R8: 1k, Resistor_SMD:R_1206_3216Metric_Pad1.30x1.75mm_HandSolder, B.Cu at (150.0, 87.8)
- added U3: CNY17-3, Package_DIP:DIP-6_W7.62mm_LongPads, F.Cu at (115.2, 100.4)
- C1: value 18p -> 100n; footprint Capacitor_SMD:C_0805_2012Metric_Pad1.18x1.45mm_HandSolder -> Capacitor_SMD:C_1206_3216Metric_Pad1.33x1.80mm_HandSolder
- C16: value 100n -> 10u
- C4: value 100n -> 18p; footprint Capacitor_SMD:C_1206_3216Metric_Pad1.33x1.80mm_HandSolder -> Capacitor_SMD:C_0805_2012Metric_Pad1.18x1.45mm_HandSolder
- J1: footprint TerminalBlock:TerminalBlock_Altech_AK300-4_P5.00mm -> Connector_Phoenix_MSTB:PhoenixContact_MSTBVA_2,5_4-G-5,08_1x04_P5.08mm_Vertical
- J4: renamed from J5; footprint Connector_PinSocket_2.54mm:PinSocket_1x07_P2.54mm_Vertical -> Connector_PinSocket_2.54mm:PinSocket_1x09_P2.54mm_Vertical
- J5: renamed from J6; footprint Connector_PinSocket_2.54mm:PinSocket_1x07_P2.54mm_Vertical -> Connector_PinSocket_2.54mm:PinSocket_1x09_P2.54mm_Vertical
- J8: renamed from J10; footprint Connector_PinSocket_2.54mm:PinSocket_1x03_P2.54mm_Vertical -> Connector_PinHeader_2.54mm:PinHeader_1x05_P2.54mm_Vertical
- R1: value 1.2M -> 10E
- R13: footprint Resistor_SMD:R_1206_3216Metric_Pad1.30x1.75mm_HandSolder -> Resistor_SMD:R_1206_3216Metric
- R14: value 10E -> 100k; footprint Resistor_SMD:R_1206_3216Metric_Pad1.30x1.75mm_HandSolder -> Resistor_SMD:R_1206_3216Metric
- R15: value 10E -> 150k; footprint Resistor_SMD:R_2816_7142Metric_Pad3.20x4.45mm_HandSolder -> Resistor_SMD:R_1206_3216Metric_Pad1.30x1.75mm_HandSolder
- R16: value 270k -> 150k
- R19: value 330E -> 180k
- R2: value 150k -> 1.2M
- R25: renamed from R26; moved to B.Cu
- R3: value 150k -> 10E; footprint Resistor_SMD:R_1206_3216Metric_Pad1.30x1.75mm_HandSolder -> Resistor_SMD:R_0805_2012Metric_Pad1.20x1.40mm_HandSolder
- R4: renamed from R22; footprint Resistor_SMD:R_1206_3216Metric_Pad1.30x1.75mm_HandSolder -> Resistor_SMD:R_0805_2012Metric_Pad1.20x1.40mm_HandSolder
- R5: renamed from R17; footprint Resistor_SMD:R_1206_3216Metric_Pad1.30x1.75mm_HandSolder -> Resistor_SMD:R_0805_2012Metric_Pad1.20x1.40mm_HandSolder
- R6: renamed from R21; footprint Resistor_SMD:R_1206_3216Metric_Pad1.30x1.75mm_HandSolder -> Resistor_SMD:R_0805_2012Metric_Pad1.20x1.40mm_HandSolder
- R7: renamed from R18; footprint Resistor_SMD:R_1206_3216Metric_Pad1.30x1.75mm_HandSolder -> Resistor_SMD:R_0805_2012Metric_Pad1.20x1.40mm_HandSolder
- U4: value LNK625PG -> LM317_TO-252; footprint Package_DIP:PowerIntegrations_PDIP-8C -> Package_TO_SOT_SMD:TO-252-2; moved to B.Cu
- moved R1 75.6 mm to (136.3, 70.4)
- moved C1 69.4 mm to (136.3, 74.6), turned to 180 degrees
- moved FB1 66.5 mm to (135.6, 67.6), turned to 180 degrees
- moved R16 65.2 mm to (164.5, 94.2)
- moved Y1 60.5 mm to (120.6, 84.0), turned to 90 degrees
- moved R19 56.2 mm to (157.9, 94.2), turned to 90 degrees
- moved C8 55.6 mm to (140.8, 77.0)
- moved C9 55.1 mm to (138.0, 78.6)
- moved R14 54.3 mm to (130.4, 76.7), turned to 180 degrees
- moved R3 53.4 mm to (130.5, 70.4), turned to 0 degrees
- moved C11 52.6 mm to (136.9, 88.6), turned to 180 degrees
- moved C2 52.3 mm to (118.5, 84.0), turned to -90 degrees
- moved R11 50.0 mm to (144.8, 75.4)
- moved C7 49.6 mm to (138.0, 84.7), turned to 90 degrees
- moved R12 49.5 mm to (144.8, 79.4)
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- renumbered J9 to J2, J8 to J3, J7 to J6, L1 to L5, R6 to R20, R7 to R21, R8 to R22
Connections:
- net /SDI renamed /MOSI
- C1 pad 1: /OSC1 -> /3V3A
- C1 pad 2: GNDD -> GNDA
- C11 pad 1: /3V3D -> GNDA
- C11 pad 2: GNDD -> Net-(U1-REFIN+/OUT)
- C12 pad 1: /3V3D -> GNDA
- C12 pad 2: GNDD -> Net-(U1-REFIN+/OUT)
- C16 pad 2: GND -> GNDD
- C2 pad 1: /OSC2 -> /OSC1
- C3 pad 1: /CH0- -> /3V3D
- C3 pad 2: GNDA -> GNDD
- C4 pad 1: GNDA -> /OSC2
- C4 pad 2: /CH0+ -> GNDD
- C5 pad 1: /CH1+ -> /3V3D
- C5 pad 2: GNDA -> GNDD
- C6 pad 1: GNDA -> /CH1+
- C6 pad 2: /CH1- -> GNDA
- C7 pad 2: Net-(U1-REFIN+/OUT) -> /CH1-
- C8 pad 1: GNDA -> /CH0+
- C8 pad 2: Net-(U1-REFIN+/OUT) -> GNDA
- C9 pad 1: /3V3A -> GNDA
- C9 pad 2: GNDA -> /CH0-
- J1 pad 1: /current_neg -> GNDD
- J1 pad 2: /HIGH_in -> HIGH_in
- J1 pad 3: /HIGH_in -> HIGH_in
- J2 pad 1: /5V -> +5V
- J4 pad 1: +3.3V -> +5V
- J4 pad 2: /XDIR/PA4 -> /CS_adc
- J4 pad 3: /PA5 -> /CS_funk
- J5 pad 1: /SDA/XCK/PB1 -> GND
- J5 pad 2: /SCL/XDIR/PB0 -> /SCK
- J5 pad 3: /RESET-UDPI -> /MISO
- J5 pad 5: /RXD/PA2 -> /RESET-UDPI
- J5 pad 6: /SCLK -> /SCL/XDIR/PB0
- J5 pad 7: GND -> /SDA/XCK/PB1
- J6 pad 1: /PA6 -> /CS_funk
- J6 pad 2: /RXD/PA2 -> /MISO
- J6 pad 4: /SCLK -> /SCK
- J6 pad 5: /PA5 -> /PA6
- J8 pad 1: /RESET-UDPI -> GND
- J8 pad 2: /RxD/PB3 -> +5V
- L3 pad 1: /current_neg -> GNDD
- L5 pad 1: /HIGH_in -> HIGH_in
- L5 pad 2: Net-(L1-Pad2) -> Net-(L5-Pad2)
- R1 pad 1: /OSC1 -> Net-(FB1-Pad1)
- R1 pad 2: /OSC2 -> /3V3A
- R10 pad 1: GNDA -> /voltage_pos
- R10 pad 2: /CH0+ -> /CH1+
- R11 pad 1: /voltage_pos -> Net-(L2-Pad2)
- R11 pad 2: /CH0- -> /CH0+
- R12 pad 1: Net-(L2-Pad2) -> Net-(L3-Pad2)
- R12 pad 2: /CH1+ -> /CH0-
- R13 pad 1: Net-(L3-Pad2) -> Net-(R13-Pad1)
- R13 pad 2: /CH1- -> /3V3D
- R14 pad 1: Net-(FB1-Pad1) -> /3V3D
- R14 pad 2: /3V3A -> /~{DR}_MCP
- R15 pad 1: /HIGH_in -> Net-(L5-Pad2)
- R15 pad 2: Net-(D4-K) -> Net-(R15-Pad2)
- R16 pad 1: Net-(C19-Pad2) -> Net-(R15-Pad2)
- R19 pad 2: Net-(C19-Pad2) -> Net-(R19-Pad2)
- R2 pad 1: Net-(L1-Pad2) -> /OSC1
- R2 pad 2: Net-(R2-Pad2) -> /OSC2
- R20 pad 1: /current_neg -> GNDD
- R21 pad 1: /current_neg -> GNDD
- R22 pad 1: Net-(R5-Pad2) -> Net-(R19-Pad2)
- R25 pad 1: /PA5 -> /SDA/XCK/PB1
- R3 pad 1: Net-(R2-Pad2) -> +3.3V
- R3 pad 2: Net-(R3-Pad2) -> /3V3D
- R9 pad 1: /voltage_pos -> GNDA
- R9 pad 2: GNDA -> /CH1-
- U1 pad 6: /CH1+ -> /CH1-
- U1 pad 7: /CH1- -> /CH1+
- U2 pad 1: +3.3V -> +5V
- U2 pad 3: /PA5 -> /CS_adc
- U2 pad 4: /SCLK -> /SCK
- U2 pad 6: /RXD/PA2 -> /MISO
- U2 pad 7: +3.3V -> +5V
- U4 pad 2: Net-(U4-BP) -> +3.3V
Routing:
- net HIGH_in: track 0.00 -> 173.9 mm
- net +5V: track 0.00 -> 146.6 mm
- net +3.3V: track 134.6 -> 37.1 mm, vias 2 -> 0
- net /PA5: track 81.0 -> 0.00 mm, vias 2 -> 0
- net Net-(L3-Pad2): track 82.6 -> 1.97 mm, vias 2 -> 0
- net Net-(L2-Pad2): track 77.8 -> 1.97 mm, vias 2 -> 0
- net /current_neg: track 71.0 -> 0.00 mm
- net /5V: track 71.0 -> 0.00 mm, vias 2 -> 0
- net Net-(R16-Pad2): track 74.5 -> 4.57 mm
- net Net-(L1-Pad2): track 69.3 -> 0.00 mm, vias 2 -> 0
- net /SCL/XDIR/PB0: track 0.38 -> 66.1 mm
- net /CS_adc: track 0.00 -> 64.8 mm, vias 0 -> 2
- net Net-(C18-Pad2): track 56.4 -> 0.00 mm
- net /SCK: track 0.00 -> 49.9 mm, vias 0 -> 2
- net /OSC1: track 62.3 -> 12.5 mm
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- added copper zone on In2.Cu, net GNDA
- added copper zone on F.Cu, net GNDD
- added copper zone on In1.Cu, net GNDD
- added copper zone on In2.Cu, net GNDD
Other:
- board text removed: "ATtiny status led"

Commit message: various fixes
Parts:
- added R26: 10E, Resistor_SMD:R_0805_2012Metric_Pad1.20x1.40mm_HandSolder, B.Cu at (122.5, 91.3)
- J5: footprint Connector_PinSocket_2.54mm:PinSocket_1x09_P2.54mm_Vertical -> Connector_PinSocket_2.54mm:PinSocket_1x07_P2.54mm_Vertical
- R1: footprint Resistor_SMD:R_1206_3216Metric_Pad1.30x1.75mm_HandSolder -> Resistor_SMD:R_0805_2012Metric_Pad1.20x1.40mm_HandSolder
- moved FB1 3.25 mm to (133.4, 70.0)
- moved J10 2.46 mm to (111.2, 97.7)
- moved J4 2.15 mm to (182.4, 139.1)
- moved J5 2.15 mm to (167.2, 139.1)
- moved R1 2.07 mm to (138.4, 70.7), turned to 180 degrees
- moved R3 2.04 mm to (128.4, 70.7)
- moved R25 1.98 mm to (171.4, 123.8)
- moved C13 1.14 mm to (155.8, 64.6)
- moved J13 0.71 mm to (107.5, 96.0)
- moved D1 0.71 mm to (121.7, 65.0)
- moved D2 0.71 mm to (121.8, 68.4)
Connections:
- U3 pad 6: /~{RESET} -> Net-(R26-Pad2)
Routing:
- net HIGH_in: track 173.9 -> 82.6 mm
- net +5V: track 146.6 -> 201.1 mm, vias 0 -> 2
- net /MOSI: track 45.8 -> 53.2 mm, vias 3 -> 1
- net Net-(U4-ADJ): track 5.40 -> 11.3 mm
- net /MISO: track 42.9 -> 46.9 mm, vias 2 -> 1
- net Net-(R26-Pad2): track 0.00 -> 3.51 mm
- net /SCK: track 49.9 -> 53.1 mm, vias 2 -> 1
- net +3.3V: track 37.1 -> 33.9 mm
- net /~{RESET}: track 30.2 -> 27.1 mm, vias 1 -> 2
- net Net-(FB1-Pad1): track 3.68 -> 5.92 mm
- net /PA6: track 23.6 -> 25.7 mm, vias 2 -> 0
- net /SCL/XDIR/PB0: track 66.1 -> 68.3 mm
- net /CS_funk: track 22.4 -> 24.6 mm, vias 2 -> 0
- net /PA7: track 22.1 -> 24.2 mm, vias 2 -> 0
- net /GPIO1: track 21.1 -> 23.2 mm, vias 2 -> 0
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
Commit message: Small changes
Parts:
- added C17: 100n, Capacitor_SMD:C_1206_3216Metric_Pad1.33x1.80mm_HandSolder, F.Cu at (26.6, 27.7)
- added C18: 10u, Capacitor_SMD:C_1206_3216Metric_Pad1.33x1.80mm_HandSolder, F.Cu at (26.6, 31.0)
- added R27: 6.8, Resistor_THT:R_Radial_Power_L12.0mm_W8.0mm_P5.00mm, F.Cu at (3.77, 30.8)
- added RV1: B72214S0551K101, Resistor_THT:R_Axial_DIN0204_L3.6mm_D1.6mm_P7.62mm_Horizontal, F.Cu at (14.5, 27.6)
- added U5: ~, Power_Supply:RS_2333523, F.Cu at (20.1, 12.8)

Commit message: SMPS routed
Parts:
- removed R13: 1k, Resistor_SMD:R_1206_3216Metric
- removed TP4: TestPoint, TestPoint:TestPoint_Plated_Hole_D3.0mm
- removed U3: CNY17-3, Package_DIP:DIP-6_W7.62mm_LongPads
- added U6: ADuM1250, Package_SO:SO-8_5.3x6.2mm_P1.27mm, B.Cu at (120.6, 111.4)
- C17, C18: moved to B.Cu
- moved U5 140.4 mm to (109.8, 120.7), turned to -90 degrees
- moved C17 134.4 mm to (111.2, 132.1), turned to -90 degrees
- moved C18 134.0 mm to (114.5, 132.1), turned to -90 degrees
- moved RV1 116.8 mm to (107.4, 98.4)
- moved R27 114.8 mm to (101.2, 91.4), turned to -90 degrees
- moved J13 75.4 mm to (181.7, 109.5)
- moved J10 67.8 mm to (177.9, 109.5)
- moved J9 40.1 mm to (157.9, 87.7)
- moved J11 4.72 mm to (180.4, 113.5), turned to -90 degrees
- moved R25 1.95 mm to (173.0, 122.7)
- moved J2 1.87 mm to (127.6, 121.7)
- moved J3 1.87 mm to (161.7, 125.2)
- moved J6 1.87 mm to (161.8, 129.0)
- moved J5 0.91 mm to (168.1, 139.1)
- moved J4 0.91 mm to (183.3, 139.1)
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Connections:
- R27 pad 1: Net-(F1-Pad1) -> HIGH_in
- RV1 pad 1: Net-(F1-Pad1) -> HIGH_in
- U5 pad 1: (no net) -> Net-(R27-Pad2)
- U5 pad 2: (no net) -> GNDD
- U5 pad 4: (no net) -> GND
- U5 pad 6: (no net) -> +5V
Routing:
- net HIGH_in: track 82.6 -> 200.7 mm
- net GNDD: track 33.3 -> 117.8 mm
- net +5V: track 201.1 -> 247.0 mm, vias 2 -> 3
- net Net-(U6-SCL2): track 3.51 -> 20.2 mm, vias 0 -> 2
- net /3V3D: track 66.0 -> 78.7 mm, vias 3 -> 4
- net GND: track 5.14 -> 13.6 mm
- net Net-(R27-Pad2): track 0.00 -> 8.29 mm
- net /SCL/XDIR/PB0: track 68.3 -> 60.0 mm, vias 0 -> 1
- net Net-(J11-Pin_2): track 16.6 -> 10.6 mm
- net /RESET-UDPI: track 33.9 -> 39.7 mm
- net Net-(R13-Pad1): track 3.31 -> 0.00 mm
- net /SDA/XCK/PB1: track 2.66 -> 3.80 mm
- net /CS_adc: track 64.8 -> 65.9 mm
- net /GPIO0: track 23.2 -> 22.2 mm
- net /GPIO1: track 23.2 -> 22.2 mm
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Other:
- board text removed: "RxD"
- board text removed: "TxD"
- board text removed: "UDPI"
